File: KiCAD/witherbone.sch (KiCad schematic (older format))
At the start: 50 parts, among them SW1 POWER, U1 OSD3358-512M-BSM, U2 SN74LVC1G07DCK, U3 TPD4S012DRY, X1 10118192-0001LF, X2 MICROSD, Y1 24 MHz

Commit message: Hack in TFP410
Parts:
- added U?: TFP410, QFP50P1200X1200X120-65N, symbol TFP410
Connections:
- net (U1.G1)LCD.D2.B5: now also U?.58 (DATA5)
- net (U1.G2)LCD.D1.B4: now also U?.59 (DATA4)
- net (U1.G3)LCD.D0.B3: now also U?.60 (DATA3)
- net (U1.H1)LCD.D5.G2: now also U?.51 (DATA10)
- net (U1.H2)LCD.D4.B7: now also U?.54 (DATA7)
- net (U1.H3)LCD.D3.B6: now also U?.55 (DATA6)
- net (U1.J1)LCD.D8.G5: now also U?.46 (DATA13)
- net (U1.J2)LCD.D7.G4: now also U?.47 (DATA12)
- net (U1.J3)LCD.D6.G3: now also U?.50 (DATA11)
- net (U1.K1)LCD.D11.R3: now also U?.40 (DATA19)
- net (U1.K2)LCD.D10.G7: now also U?.44 (DATA15)
- net (U1.K3)LCD.D9.G6: now also U?.45 (DATA14)
- net (U1.L1)LCD.D14.R6: now also U?.37 (DATA22)
- net (U1.L2)LCD.D13.R5: now also U?.38 (DATA21)
- net (U1.L3)LCD.D12.R4: now also U?.39 (DATA20)
- net (U1.M3)LCD.D15.R7: now also U?.36 (DATA23)
Other:
- note added: "Based on PocketBeagle (https://beagleboard.org/pocket)"
- note added: "Witherbone\n"
- note removed: "Pocket Beagle\n"
- note removed: "https://beagleboard.org/pocket"
- moved on the sheet: U1D
