File: EAGLE/whitherbone.brd (EAGLE design)
At the start: 86.4 x 54.6 mm, 225 parts, among them IC10 TXS0108ERGYR, IC11 TXS0108ERGYR, IC12 TPS2051BDGN, IC13 SN74AUC1G74, IC14 TPD4S012DRY, IC15 TPD4S012DRY, IC17 SN74LVC2G241DCUR, IC18 TL1963ADCQR, IC19 AP2112K-1.8TRG1 3.3V, IC2 SN74LVC1G07DCK, IC4 7805T, IC7 IP4283CZ10-TBR, IC8 IP4283CZ10-TBR, IC9 TDA19988BHN/C1,557, J1 1-1747981-1, Q2 32.768kHz, Q4 24 MHz, T3 BSS138W-7-F, T4 BSS138W-7-F, U1 OSD3358-512M-BSM, X2 SCHA5B0200, X4 10118192-0001LF

Commit message: USR LED connections
Connections:
- removed net VIN_USB: U1.R9, U1.T9
- net I2C0_SCL: now also U1.C10, U1.D10
- net I2C0_SDA: now also U1.C11, U1.D11
- net PWR_BUT: now also U1.T11
- net USB_DC: now also U1.R9, U1.T9
- net USR0: now also U1.P13
- net USR1: now also U1.T14
- net USR2: now also U1.R14
- net USR3: now also U1.P14
Changed lines of the file:
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@@
 <wire x1="20.566" y1="6.604" x2="20.566" y2="7.485" width="0.1524" layer="1"/>
 <wire x1="20.566" y1="7.485" x2="20.825" y2="7.744" width="0.1524" layer="1"/>
+<contactref element="U1" pad="C11"/>
+<contactref element="U1" pad="D11"/>
+<wire x1="45.5168" y1="73.7616" x2="46.7868" y2="73.7616" width="0" layer="19" extent="1-1"/>
+<wire x1="79.15" y1="32.5" x2="46.7868" y2="73.7616" width="0" layer="19" extent="1-1"/>
 <wire x1="20.825" y1="7.744" x2="21.656" y2="8.448" width="0" layer="19" extent="1-1"/>
 </signal>
@@
 <wire x1="20.566" y1="12.192" x2="20.566" y2="11.311" width="0.1524" layer="1"/>
 <wire x1="20.566" y1="11.311" x2="20.825" y2="11.052" width="0.1524" layer="1"/>
-<wire x1="21.656" y1="10.348" x2="20.825" y2="11.052" width="0" layer="19" extent="1-1"/>
+<contactref element="U1" pad="C10"/>
+<contactref element="U1" pad="D10"/>
+<wire x1="45.5168" y1="72.4916" x2="46.7868" y2="72.4916" width="0" layer="19" extent="1-1"/>
+<wire x1="79.15" y1="33" x2="46.7868" y2="72.4916" width="0" layer="19" extent="1-1"/>
+<wire x1="20.825" y1="11.052" x2="21.656" y2="10.348" width="0" layer="19" extent="1-1"/>
 </signal>
 <signal name="USB.CLIENT.D-">
@@
 <wire x1="53.721" y1="36.195" x2="54.356" y2="35.56" width="0.8128" layer="2"/>
 <contactref element="U1" pad="P9"/>
+<contactref element="U1" pad="R9"/>
+<contactref element="U1" pad="T9"/>
+<wire x1="60.7568" y1="71.2216" x2="62.0268" y2="71.2216" width="0" layer="19" extent="1-1"/>
+<wire x1="59.4868" y1="71.2216" x2="60.7568" y2="71.2216" width="0" layer="19" extent="1-1"/>
 <wire x1="53.721" y1="36.195" x2="59.4868" y2="71.2216" width="0" layer="19" extent="1-2"/>
 <wire x1="7.753" y1="44.077" x2="10.279" y2="45.974" width="0" layer="19" extent="1-1"/>
@@
 <wire x1="27.9654" y1="7.5438" x2="28.2702" y2="7.239" width="0.1524" layer="14"/>
 <wire x1="28.2702" y1="7.239" x2="30.1752" y2="7.239" width="0.1524" layer="14"/>
+<contactref element="U1" pad="T11"/>
+<wire x1="9.9375" y1="42.66" x2="62.0268" y2="73.7616" width="0" layer="19" extent="1-1"/>
 </signal>
 <signal name="VDD_3V3B">
@@
 <wire x1="16.764" y1="47.7774" x2="12.9286" y2="47.7774" width="0.1524" layer="16"/>
 <wire x1="12.9286" y1="47.7774" x2="9.017" y2="51.689" width="0.1524" layer="16"/>
+<contactref element="U1" pad="P13"/>
+<wire x1="35.2044" y1="48.0822" x2="59.4868" y2="76.3016" width="0" layer="19" extent="1-16"/>
 </signal>
 <signal name="USR1">
@@
 <wire x1="9.7536" y1="49.0728" x2="9.3345" y2="49.4919" width="0.1524" layer="16"/>
 <wire x1="9.3345" y1="49.4919" x2="9.3345" y2="49.9745" width="0.1524" layer="16"/>
+<contactref element="U1" pad="T14"/>
+<wire x1="34.8996" y1="47.4726" x2="62.0268" y2="77.5716" width="0" layer="19" extent="1-16"/>
 </signal>
 <signal name="USR2">
@@
 <wire x1="10.5918" y1="48.768" x2="9.525" y2="48.768" width="0.1524" layer="16"/>
 <wire x1="9.525" y1="48.768" x2="8.636" y2="49.657" width="0.1524" layer="16"/>
+<contactref element="U1" pad="R14"/>
+<wire x1="34.7472" y1="47.1678" x2="60.7568" y2="77.5716" width="0" layer="19" extent="1-16"/>
 </signal>
 <signal name="USR3">
@@
 <wire x1="12.8016" y1="47.4726" x2="10.6172" y2="49.657" width="0.1524" layer="16"/>
 <wire x1="10.6172" y1="49.657" x2="10.033" y2="49.657" width="0.1524" layer="16"/>
+<contactref element="U1" pad="P14"/>
+<wire x1="35.052" y1="47.7774" x2="59.4868" y2="77.5716" width="0" layer="19" extent="1-16"/>
 </signal>
 <signal name="N$34">
@@
 <contactref element="U1" pad="H9"/>
 </signal>
-<signal name="VIN_USB">
-<contactref element="U1" pad="R9"/>
-<contactref element="U1" pad="T9"/>
-<wire x1="60.7568" y1="71.2216" x2="62.0268" y2="71.2216" width="0" layer="19" extent="1-1"/>
-</signal>
 <signal name="N$10">

Commit message: Power and other clean-up
Parts:
- removed C18: .1uF, 6.3V, rcl:C0402K
- removed R40: 10k, 1%, rcl:R0402
- removed R41, R42: 1.5k, 1%, rcl:R0402
- removed R54: 0, 1%, rcl:R0402
- added BT1: LTST-C191TBKT, GHI-BasicComponents:0603-LED
- added R9: 1k, rcl:R0402
- added T1: BSS138W-7-F, GHI Transistors:SOT-323(DIODES)
Connections:
- removed net GPIO1_16: R54.1
- removed net GPIO1_16.SIP: R54.2
- removed net GPIO3_21: R110.2
- removed net HDMICLK_DIS#: OSC1.1
- removed net N$54: R40.2, TP1.P$1
- removed net SPI1_CS0: IC9.25
- removed net SPI1_D0: IC9.24
- removed net SPI1_SCLK: IC9.23
- new net EEPROM_WP: TP1.P$1, U1.M2, U1.N3
- new net HDMI_AUDBCLK: IC9.23, U1.A1
- new net HDMI_AUDCLK: R110.2, U1.C4
- new net HDMI_AUDCLK_DIS#: OSC1.1, U1.T16
- new net HDMI_AUDDOUT: IC9.25, U1.B1
- new net HDMI_AUDWCLK: IC9.24, U1.A2
- new net N$2: BT1.A, R9.1
- new net N$21: U1.N10, U1.N11
- new net N$23: U1.N4, U1.N5
- new net N$26: U1.L4, U1.M4
- new net N$27: U1.D4, U1.E4
- new net N$8: BT1.K, T1.D
- new net VDD_RTC: U1.L11
- new net WIFI_LED(GPIO3_01): T1.G, U1.F14
- net 3.3V-WIFI: now also R9.2
- net GND: now also T1.S; no longer C18.2
- net HDMI_INT: now also U1.T15
- net I2C0_SCL: no longer R41.2
- net I2C0_SDA: no longer R42.2
- net SYS_5V: now also U1.L6, U1.L7
- net SYS_RTC_1P8V: no longer U1.L11
- net SYS_VDD1_3P3V: no longer U1.F7, U1.G7
- net SYS_VDD2_3P3V: no longer U1.G11
- net SYS_VOUT: no longer U1.L6, U1.L7
- net USB1_OC#: now also U1.R15
- net VDD_3V3AUX: now also U1.G11
- net VDD_3V3B: now also U1.F7, U1.G7; no longer C18.1, R40.1, R41.1, R42.1
Routing:
- net SPI1_CS0: track 48.1 -> 0.00 mm, vias 1 -> 0
- net HDMI_AUDDOUT: track 0.00 -> 48.1 mm, vias 0 -> 1
- net SPI1_D0: track 45.8 -> 0.00 mm, vias 1 -> 0
- net HDMI_AUDWCLK: track 0.00 -> 45.8 mm, vias 0 -> 1
- net GPIO1_16: track 44.8 -> 0.00 mm, vias 1 -> 0
- net SPI1_SCLK: track 41.3 -> 0.00 mm, vias 1 -> 0
- net HDMI_AUDBCLK: track 0.00 -> 41.3 mm, vias 0 -> 1
- net HDMI_AUDCLK: track 0.00 -> 25.9 mm, vias 0 -> 2
- net GPIO3_21: track 25.9 -> 0.00 mm, vias 2 -> 0
- net HDMI_AUDCLK_DIS#: track 0.00 -> 19.9 mm, vias 0 -> 2
- net HDMICLK_DIS#: track 19.9 -> 0.00 mm, vias 2 -> 0
- net N$54: track 6.02 -> 0.00 mm
- net EEPROM_WP: track 0.00 -> 3.48 mm
- net GPIO1_16.SIP: track 1.79 -> 0.00 mm, vias 1 -> 0
- net I2C0_SDA: track 98.8 -> 97.5 mm
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
Commit message: Power and other clean-up
Parts:
- removed FB7: 1k BLM15AG102SN1D, rcl:R0402
- removed R14: 0, 1%, rcl:R0402
Connections:
- removed net SYS_RTC_1P8V: U1.K11
- removed net SYS_VDD1_3P3V: U1.F6, U1.G6
- removed net SYS_VDD2_3P3V: U1.F11
- removed net SYS_VOUT: U1.K6, U1.K7
- net CLKOUT2: no longer FB7.1, R14.1
- net N$28: now also U1.A7, U1.B7; no longer R14.2
- net N$29: now also U1.A9, U1.B9; no longer FB7.2
- net PMIC_PGOOD: now also U1.N12, U1.P11
- net SYS_5V: now also U1.K6, U1.K7
- net SYS_RESET#: now also U1.R11
- net VDD_3V3AUX: now also U1.F11
- net VDD_3V3B: now also U1.F6, U1.G6
- net VDD_RTC: now also U1.K11
Routing:
- net N$29: track 23.7 -> 0.00 mm, vias 2 -> 0
- net N$28: track 23.2 -> 0.00 mm, vias 2 -> 0
- net CLKOUT2: track 65.0 -> 60.2 mm
Changed lines of the file:
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@@
 <attribute name="VALUE" x="30.623" y="9.784" size="1.016" layer="27"/>
 </element>
-<element name="R14" library="rcl" package="R0402" value="0, 1%" x="68.58" y="6.858" smashed="yes" rot="MR90">
-<attribute name="NAME" x="68.5292" y="8.0264" size="0.8128" layer="26" ratio="15" rot="MR90" align="center-left"/>
-<attribute name="VALUE" x="66.548" y="5.969" size="1.27" layer="28" rot="MR90"/>
-</element>
-<element name="FB7" library="rcl" package="R0402" value="1k BLM15AG102SN1D" x="67.31" y="6.858" smashed="yes" rot="MR90">
-<attribute name="NAME" x="67.1576" y="7.9248" size="0.8128" layer="26" ratio="15" rot="MR90" align="center-left"/>
-<attribute name="VALUE" x="65.278" y="5.969" size="1.27" layer="28" rot="MR90"/>
-</element>
 <element name="C27" library="rcl" package="C0402K" value="47pF, 6.3V" x="55.88" y="47.498" smashed="yes" rot="MR270">
 <attribute name="NAME" x="66.929" y="39.497" size="0.8128" layer="26" ratio="15" rot="MR0" align="center-left"/>
@@
 <contactref element="U1" pad="F7"/>
 <contactref element="U1" pad="G7"/>
+<contactref element="U1" pad="F6"/>
+<contactref element="U1" pad="G6"/>
 <wire x1="80.4" y1="29.75" x2="84.447" y2="33.909" width="0" layer="19" extent="1-1"/>
 <wire x1="79.375" y1="19.812" x2="79.4004" y2="29.4132" width="0" layer="19" extent="1-1"/>
@@
 <wire x1="59.055" y1="47.633" x2="69.85" y2="46.998" width="0" layer="19" extent="1-16"/>
 <wire x1="68.3514" y1="28.7274" x2="79.4004" y2="29.4132" width="0" layer="19" extent="16-16"/>
-<wire x1="50.5968" y1="68.6816" x2="51.943" y2="51.435" width="0" layer="19" extent="1-16"/>
+<wire x1="50.5968" y1="67.4116" x2="51.943" y2="51.435" width="0" layer="19" extent="1-16"/>
+<wire x1="50.5968" y1="68.6816" x2="50.5968" y2="67.4116" width="0" layer="19" extent="1-1"/>
 <wire x1="49.3268" y1="68.6816" x2="50.5968" y2="68.6816" width="0" layer="19" extent="1-1"/>
+<wire x1="49.3268" y1="67.4116" x2="50.5968" y2="67.4116" width="0" layer="19" extent="1-1"/>
 <wire x1="38.735" y1="32.004" x2="46.228" y2="49.403" width="0" layer="19" extent="16-16"/>
 <wire x1="38.735" y1="30.988" x2="38.735" y2="32.004" width="0" layer="19" extent="1-1"/>
@@
 <wire x1="31.623" y1="8.9154" x2="32.1056" y2="9.398" width="0.1524" layer="1"/>
 <wire x1="32.1056" y1="9.398" x2="32.723" y2="9.398" width="0.1524" layer="1"/>
+<contactref element="U1" pad="N12"/>
+<contactref element="U1" pad="P11"/>
+<wire x1="58.2168" y1="75.0316" x2="59.4868" y2="73.7616" width="0" layer="19" extent="1-1"/>
+<wire x1="45.466" y1="11.176" x2="59.4868" y2="73.7616" width="0" layer="19" extent="1-1"/>
 </signal>
 <signal name="VDD_3V3AUX">
@@
 <wire x1="50.3682" y1="36.4998" x2="51.562" y2="35.306" width="0.254" layer="14"/>
 <contactref element="U1" pad="G11"/>
-<wire x1="36.4998" y1="46.5582" x2="50.5968" y2="73.7616" width="0" layer="19" extent="1-14"/>
+<contactref element="U1" pad="F11"/>
+<wire x1="49.3268" y1="73.7616" x2="50.5968" y2="73.7616" width="0" layer="19" extent="1-1"/>
+<wire x1="36.4998" y1="46.5582" x2="49.3268" y2="73.7616" width="0" layer="19" extent="1-14"/>
 </signal>
 <signal name="JTAG_TRSTN">
@@
 </signal>
 <signal name="CLKOUT2">
-<contactref element="FB7" pad="1"/>
-<contactref element="R14" pad="1"/>
-<wire x1="67.31" y1="6.358" x2="68.58" y2="6.358" width="0.1524" layer="16"/>
-<wire x1="69.215" y1="5.723" x2="69.215" y2="3.175" width="0.1524" layer="16"/>
 <wire x1="38.354" y1="16.764" x2="39.116" y2="17.526" width="0.1524" layer="16"/>
 <via x="39.116" y="17.526" extent="1-16" drill="0.4064"/>
@@
 <wire x1="66.8274" y1="7.4676" x2="69.215" y2="5.08" width="0.1524" layer="14"/>
 <wire x1="69.215" y1="5.08" x2="69.215" y2="3.175" width="0.1524" layer="14"/>
-<wire x1="69.215" y1="5.723" x2="68.58" y2="6.358" width="0.1524" layer="16"/>
 <contactref element="IC11" pad="16"/>
 <wire x1="39.116" y1="17.526" x2="39.116" y2="18.034" width="0.1524" layer="16"/>
@@
 <wire x1="29.718" y1="24.765" x2="34.036" y2="20.447" width="0.1524" layer="14"/>
 <wire x1="34.036" y1="20.447" x2="36.703" y2="20.447" width="0.1524" layer="14"/>
-<wire x1="69.215" y1="3.175" x2="69.215" y2="3.175" width="0" layer="19" extent="14-16"/>
 </signal>
 <signal name="N$3">
@@
 <wire x1="29.202" y1="9.398" x2="29.852" y2="10.048" width="0.1524" layer="1"/>
 <wire x1="29.852" y1="10.048" x2="30.523" y2="10.048" width="0.1524" layer="1"/>
+<contactref element="U1" pad="R11"/>
+<wire x1="32.0802" y1="48.768" x2="60.7568" y2="73.7616" width="0" layer="19" extent="1-3"/>
 <wire x1="28.575" y1="5.715" x2="31.8516" y2="6.4516" width="0" layer="19" extent="1-3"/>
 </signal>
-<signal name="N$28">
-<contactref element="R14" pad="2"/>
-<via x="49.276" y="13.843" extent="1-16" drill="0.4064"/>
-<wire x1="49.149" y1="13.843" x2="49.276" y2="13.843" width="0.1524" layer="1"/>
-<wire x1="49.276" y1="13.843" x2="49.8856" y2="13.2334" width="0.1524" layer="14"/>
-<wire x1="49.8856" y1="13.2334" x2="57.3024" y2="13.2334" width="0.1524" layer="14"/>
-<wire x1="57.3024" y1="13.2334" x2="57.6072" y2="13.5382" width="0.1524" layer="14"/>
-<wire x1="57.6072" y1="13.5382" x2="63.881" y2="13.5382" width="0.1524" layer="14"/>
-<via x="67.945" y="9.271" extent="1-16" drill="0.4064"/>
-<wire x1="68.58" y1="7.358" x2="68.58" y2="8.636" width="0.1524" layer="16"/>
-<wire x1="68.58" y1="8.636" x2="67.945" y2="9.271" width="0.1524" layer="16"/>
-<wire x1="63.881" y1="13.5382" x2="67.945" y2="9.4742" width="0.1524" layer="14"/>
-<wire x1="67.945" y1="9.4742" x2="67.945" y2="9.271" width="0.1524" layer="14"/>
-</signal>
-<signal name="N$29">
-<contactref element="FB7" pad="2"/>
-<via x="48.006" y="13.843" extent="1-16" drill="0.4064"/>
-<wire x1="47.879" y1="13.843" x2="48.006" y2="13.843" width="0.1524" layer="1"/>
-<wire x1="48.006" y1="13.843" x2="48.9204" y2="12.9286" width="0.1524" layer="14"/>
-<wire x1="48.9204" y1="12.9286" x2="57.4548" y2="12.9286" width="0.1524" layer="14"/>
-<wire x1="57.4548" y1="12.9286" x2="57.7596" y2="13.2334" width="0.1524" layer="14"/>
-<wire x1="57.7596" y1="13.2334" x2="63.7286" y2="13.2334" width="0.1524" layer="14"/>
-<via x="66.929" y="9.271" extent="1-16" drill="0.4064"/>
-<wire x1="67.31" y1="7.358" x2="67.31" y2="8.89" width="0.1524" layer="16"/>
-<wire x1="67.31" y1="8.89" x2="66.929" y2="9.271" width="0.1524" layer="16"/>
-<wire x1="63.7286" y1="13.2334" x2="66.929" y2="10.033" width="0.1524" layer="14"/>
-<wire x1="66.929" y1="10.033" x2="66.929" y2="9.271" width="0.1524" layer="14"/>
-</signal>
 <signal name="USR0">
 <via x="46.736" y="32.766" extent="1-16" drill="0.4064" diameter="0.254"/>
@@
 <contactref element="U1" pad="L6"/>
 <contactref element="U1" pad="L7"/>
+<contactref element="U1" pad="K6"/>
+<contactref element="U1" pad="K7"/>
+<wire x1="54.4068" y1="68.6816" x2="55.6768" y2="68.6816" width="0" layer="19" extent="1-1"/>
 <wire x1="55.6768" y1="67.4116" x2="55.6768" y2="68.6816" width="0" layer="19" extent="1-1"/>
+<wire x1="54.4068" y1="67.4116" x2="54.4068" y2="68.6816" width="0" layer="19" extent="1-1"/>
 <wire x1="55.3974" y1="40.2336" x2="55.6768" y2="67.4116" width="0" layer="19" extent="1-15"/>
 <wire x1="74.93" y1="15.748" x2="69.088" y2="14.043" width="0" layer="19" extent="1-1"/>
@@
 <wire x1="23.6982" y1="40.2336" x2="24.003" y2="39.9288" width="0.254" layer="3"/>
 </signal>
-<signal name="SYS_RTC_1P8V">
-<contactref element="U1" pad="K11"/>
-</signal>
-<signal name="SYS_VDD1_3P3V">
-<contactref element="U1" pad="F6"/>
-<contactref element="U1" pad="G6"/>
-<wire x1="50.5968" y1="67.4116" x2="49.3268" y2="67.4116" width="0" layer="19" extent="1-1"/>
-</signal>
-<signal name="SYS_VDD2_3P3V">
-<contactref element="U1" pad="F11"/>
-</signal>
 <signal name="SYS_VDD3_3P3V">
 <contactref element="U1" pad="F8"/>
@@
 <wire x1="55.6768" y1="72.4916" x2="54.4068" y2="72.4916" width="0" layer="19" extent="1-1"/>
 </signal>
-<signal name="SYS_VOUT">
-<contactref element="U1" pad="K6"/>
-<contactref element="U1" pad="K7"/>
-<wire x1="54.4068" y1="67.4116" x2="54.4068" y2="68.6816" width="0" layer="19" extent="1-1"/>
-</signal>
 <signal name="VDDSHV1">
 <contactref element="U1" pad="J9"/>
@@
 <signal name="VDD_RTC">
 <contactref element="U1" pad="L11"/>
+<contactref element="U1" pad="K11"/>
+<wire x1="54.4068" y1="73.7616" x2="55.6768" y2="73.7616" width="0" layer="19" extent="1-1"/>
 </signal>
 <signal name="HDMI_AUDCLK">
@@
 <wire x1="51.816" y1="17.526" x2="45.5168" y2="64.8716" width="0" layer="19" extent="1-16"/>
 </signal>
+<signal name="N$28">
+<contactref element="U1" pad="A7"/>
+<contactref element="U1" pad="B7"/>
+<wire x1="42.9768" y1="68.6816" x2="44.2468" y2="68.6816" width="0" layer="19" extent="1-1"/>
+</signal>
+<signal name="N$29">
+<contactref element="U1" pad="A9"/>
+<contactref element="U1" pad="B9"/>
+<wire x1="42.9768" y1="71.2216" x2="44.2468" y2="71.2216" width="0" layer="19" extent="1-1"/>
+</signal>
 </signals>

Commit message: Stopping for the night
Parts:
- added U2: A3967SLBTR, A3967SLBTR:SOIC24WIDE
Connections:
- new net N$30: R9.2
- new net VCC: U2.14
- net 3.3V-WIFI: no longer R9.2
- net GND: now also U2.18, U2.19, U2.6, U2.7
Changed lines of the file:
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@@
 <element name="R9" library="rcl" package="R0402" value="1k" x="-36.7538" y="-78.359"/>
 <element name="T1" library="GHI Transistors" package="SOT-323(DIODES)" value="BSS138W-7-F" x="-30.861" y="-72.0344"/>
+<element name="U2" library="A3967SLBTR" package="SOIC24WIDE" value="A3967SLBTR" x="-45.72" y="-72.5678">
+<attribute name="DESCRIPTION" value=" Ic Motor Driver Pwm Full 24soic - A3967slbtr-t " x="-45.72" y="-72.5678" size="1.778" layer="27" display="off"/>
+<attribute name="DIGI-KEY_PART_NUMBER" value="620-1140-1-ND" x="-45.72" y="-72.5678" size="1.778" layer="27" display="off"/>
+<attribute name="DIGI-KEY_PURCHASE_URL" value="https://www.digikey.com/product-detail/en/allegro-microsystems-llc/A3967SLBTR-T/620-1140-1-ND/1090383?utm_source=snapeda&amp;utm_medium=aggregator&amp;utm_campaign=symbol" x="-45.72" y="-72.5678" size="1.778" layer="27" display="off"/>
+<attribute name="MF" value="Allegro" x="-45.72" y="-72.5678" size="1.778" layer="27" display="off"/>
+<attribute name="MP" value="A3967SLBTR-T" x="-45.72" y="-72.5678" size="1.778" layer="27" display="off"/>
+<attribute name="PACKAGE" value="SOIC-24 Allegro MicroSystems LLC" x="-45.72" y="-72.5678" size="1.778" layer="27" display="off"/>
+</element>
 </elements>
 <signals>
@@
 <contactref element="J1" pad="12"/>
 <contactref element="T1" pad="S"/>
+<contactref element="U2" pad="6"/>
+<contactref element="U2" pad="7"/>
+<contactref element="U2" pad="18"/>
+<contactref element="U2" pad="19"/>
 <wire x1="56.9468" y1="73.7616" x2="56.9468" y2="75.0316" width="0" layer="19" extent="1-1"/>
 <wire x1="56.9468" y1="72.4916" x2="56.9468" y2="73.7616" width="0" layer="19" extent="1-1"/>
@@
 <wire x1="-32.8798" y1="-50.845" x2="-31.3798" y2="-50.845" width="0" layer="19" extent="1-1"/>
 <wire x1="-25.3798" y1="-50.845" x2="-26.8798" y2="-50.845" width="0" layer="19" extent="1-1"/>
-<wire x1="-30.211" y1="-72.9844" x2="-29.8798" y2="-50.845" width="0" layer="19" extent="1-1"/>
+<wire x1="-45.085" y1="-67.5386" x2="-32.8798" y2="-50.845" width="0" layer="19" extent="1-1"/>
+<wire x1="-46.355" y1="-67.5386" x2="-45.085" y2="-67.5386" width="0" layer="19" extent="1-1"/>
+<wire x1="-46.355" y1="-77.597" x2="-46.355" y2="-67.5386" width="0" layer="19" extent="1-1"/>
+<wire x1="-45.085" y1="-77.597" x2="-46.355" y2="-77.597" width="0" layer="19" extent="1-1"/>
+<wire x1="-30.211" y1="-72.9844" x2="-45.085" y2="-77.597" width="0" layer="19" extent="1-1"/>
 </signal>
 <signal name="N$6">
@@
 <wire x1="29.25" y1="25.2876" x2="27.9654" y2="24.003" width="0.4064" layer="3"/>
 <wire x1="27.9654" y1="24.003" x2="27.9654" y2="23.5458" width="0.4064" layer="3"/>
-<contactref element="R9" pad="2"/>
-<wire x1="14.6" y1="16.8" x2="-36.2538" y2="-78.359" width="0" layer="19" extent="1-1"/>
+<wire x1="29.083" y1="46.355" x2="29.472" y2="47.371" width="0" layer="19" extent="1-1"/>
 <wire x1="28.872" y1="45.4" x2="28.9814" y2="46.355" width="0" layer="19" extent="1-3"/>
-<wire x1="29.472" y1="47.371" x2="29.083" y2="46.355" width="0" layer="19" extent="1-1"/>
 <wire x1="28.872" y1="43.5" x2="28.872" y2="45.4" width="0" layer="19" extent="1-1"/>
 <wire x1="26.035" y1="46.966" x2="28.9814" y2="46.355" width="0" layer="19" extent="1-3"/>
@@
 <wire x1="42.9768" y1="71.2216" x2="44.2468" y2="71.2216" width="0" layer="19" extent="1-1"/>
 </signal>
+<signal name="N$30">
+<contactref element="R9" pad="2"/>
+</signal>
+<signal name="VCC">
+<contactref element="U2" pad="14"/>
+</signal>
 </signals>
