File: EAGLE/whitherbone.sch (EAGLE design)
At the start: 224 parts, among them IC10 TXS0108ERGYR, IC11 TXS0108ERGYR, IC12 TPS2051BDGN, IC13 SN74AUC1G74, IC14 TPD4S012DRY, IC15 TPD4S012DRY, IC17 SN74LVC2G241DCUR, IC18 TL1963ADCQR, IC19 AP2112K-1.8TRG1 3.3V, IC2 SN74LVC1G07DCK, IC4 7805T, IC7 IP4283CZ10-TBR, IC8 IP4283CZ10-TBR, IC9 TDA19988BHN/C1,557, Q2 32.768kHz, Q4 24 MHz, T3 BSS138W-7-F, T4 BSS138W-7-F, U1 OSD3358-512M-BSM, X2 SCHA5B0200, X4 10118192-0001LF

Commit message: Connected WiFi/BT
Connections:
- net XDMA_EVENT_INTRO renamed XDMA_EVENT_INTR0
- net N$3: now also U1C.XDMA_EVENT_INTR0
- net SD.CD: now also U1C.SPI0_CS1
- net SD.CLK: now also U1C.MMC0_CLK
- net SD.CMD: now also U1C.MMC0_CMD
- net SD.D0: now also U1C.MMC0_DAT0
- net SD.D1: now also U1C.MMC0_DAT1
- net SD.D2: now also U1C.MMC0_DAT2
- net SD.D3: now also U1C.MMC0_DAT3
- net UART0_RXD: now also U1C.UART0_RXD
- net UART0_TXD: now also U1C.UART0_TXD
Other:
- moved on the sheet: C48, C49, FB5, FB6, IC13, IC17, R123, U1C, X1

Commit message: Connected WiFi/BT
Connections:
- net BT_EN.SIP: now also U1D.MII1_TXD0
- net BT_HCI_CTS.SIP: now also U1D.MDIO
- net BT_HCI_RTS.SIP: now also U1D.MDC
- net BT_HCI_RX.SIP: now also U1D.MII1_RXD3
- net BT_HCI_TX.SIP: now also U1D.MII1_RXD2
- net LS_BUF_OE: now also U1D.MII1_RX_CLK
- net MCU.LCD.CLK: now also U1D.LCD_PCLK
- net MCU.LCD.EN: now also U1D.LCD_AC_BIAS_EN
- net MCU.LCD.HS: now also U1D.LCD_HSYNC
- net MCU.LCD.VS: now also U1D.LCD_VSYNC
- net WL_EN.SIP: now also U1D.MII1_TX_CLK
- net WL_IRQ.SIP: now also U1D.MII1_TXD1
- net WL_SDIO_CLK.SIP: now also U1D.MII1_RXD1
- net WL_SDIO_CMD.SIP: now also U1D.MII1_TX_EN
- net WL_SDIO_D0.SIP: now also U1D.MII1_RX_DV
- net WL_SDIO_D1.SIP: now also U1D.MII1_TXD3
- net WL_SDIO_D2.SIP: now also U1D.MII1_TXD2
- net WL_SDIO_D3.SIP: now also U1D.MII1_COL
Changed lines of the file:
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@@
 <wire x1="441.96" y1="480.06" x2="416.56" y2="480.06" width="0.1524" layer="91"/>
 <label x="416.56" y="480.06" size="1.778" layer="95"/>
+<pinref part="U1" gate="D" pin="MII1_RX_CLK"/>
 </segment>
 <segment>
@@
 <wire x1="441.96" y1="472.44" x2="416.56" y2="472.44" width="0.1524" layer="91"/>
 <label x="416.56" y="472.44" size="1.778" layer="95"/>
+<pinref part="U1" gate="D" pin="MII1_RXD2"/>
 </segment>
 <segment>
@@
 <wire x1="441.96" y1="469.9" x2="416.56" y2="469.9" width="0.1524" layer="91"/>
 <label x="416.56" y="469.9" size="1.778" layer="95"/>
+<pinref part="U1" gate="D" pin="MII1_RXD3"/>
 </segment>
 <segment>
@@
 <wire x1="441.96" y1="457.2" x2="416.56" y2="457.2" width="0.1524" layer="91"/>
 <label x="416.56" y="457.2" size="1.778" layer="95"/>
+<pinref part="U1" gate="D" pin="MDC"/>
 </segment>
 <segment>
@@
 <wire x1="441.96" y1="454.66" x2="416.56" y2="454.66" width="0.1524" layer="91"/>
 <label x="416.56" y="454.66" size="1.778" layer="95"/>
+<pinref part="U1" gate="D" pin="MDIO"/>
 </segment>
 <segment>
@@
 <wire x1="502.92" y1="459.74" x2="525.78" y2="459.74" width="0.1524" layer="91"/>
 <label x="505.46" y="459.74" size="1.778" layer="95"/>
+<pinref part="U1" gate="D" pin="LCD_PCLK"/>
 </segment>
 </net>
@@
 <wire x1="502.92" y1="457.2" x2="525.78" y2="457.2" width="0.1524" layer="91"/>
 <label x="505.46" y="457.2" size="1.778" layer="95"/>
+<pinref part="U1" gate="D" pin="LCD_VSYNC"/>
 </segment>
 </net>
@@
 <wire x1="502.92" y1="454.66" x2="525.78" y2="454.66" width="0.1524" layer="91"/>
 <label x="505.46" y="454.66" size="1.778" layer="95"/>
+<pinref part="U1" gate="D" pin="LCD_HSYNC"/>
 </segment>
 </net>
@@
 <wire x1="502.92" y1="452.12" x2="525.78" y2="452.12" width="0.1524" layer="91"/>
 <label x="505.46" y="452.12" size="1.778" layer="95"/>
+<pinref part="U1" gate="D" pin="LCD_AC_BIAS_EN"/>
 </segment>
 </net>
@@
 <wire x1="441.96" y1="464.82" x2="416.56" y2="464.82" width="0.1524" layer="91"/>
 <label x="416.56" y="464.82" size="1.778" layer="95"/>
+<pinref part="U1" gate="D" pin="MII1_RX_DV"/>
 </segment>
 <segment>
@@
 <wire x1="441.96" y1="492.76" x2="416.56" y2="492.76" width="0.1524" layer="91"/>
 <label x="416.56" y="492.76" size="1.778" layer="95"/>
+<pinref part="U1" gate="D" pin="MII1_TXD3"/>
 </segment>
 <segment>
@@
 <wire x1="441.96" y1="495.3" x2="416.56" y2="495.3" width="0.1524" layer="91"/>
 <label x="416.56" y="495.3" size="1.778" layer="95"/>
+<pinref part="U1" gate="D" pin="MII1_TXD2"/>
 </segment>
 <segment>
@@
 <wire x1="441.96" y1="485.14" x2="416.56" y2="485.14" width="0.1524" layer="91"/>
 <label x="416.56" y="485.14" size="1.778" layer="95"/>
+<pinref part="U1" gate="D" pin="MII1_COL"/>
 </segment>
 <segment>
@@
 <label x="416.56" y="474.98" size="1.778" layer="95"/>
 <wire x1="441.96" y1="474.98" x2="416.56" y2="474.98" width="0.1524" layer="91"/>
+<pinref part="U1" gate="D" pin="MII1_RXD1"/>
 </segment>
 <segment>
@@
 <label x="416.56" y="490.22" size="1.778" layer="95"/>
 <wire x1="441.96" y1="490.22" x2="416.56" y2="490.22" width="0.1524" layer="91"/>
+<pinref part="U1" gate="D" pin="MII1_TX_EN"/>
 </segment>
 <segment>
@@
 <label x="416.56" y="502.92" size="1.778" layer="95"/>
 <wire x1="441.96" y1="502.92" x2="416.56" y2="502.92" width="0.1524" layer="91"/>
+<pinref part="U1" gate="D" pin="MII1_TX_CLK"/>
 </segment>
 <segment>
@@
 <label x="416.56" y="500.38" size="1.778" layer="95"/>
 <wire x1="441.96" y1="500.38" x2="416.56" y2="500.38" width="0.1524" layer="91"/>
+<pinref part="U1" gate="D" pin="MII1_TXD0"/>
 </segment>
 </net>
@@
 <wire x1="441.96" y1="497.84" x2="416.56" y2="497.84" width="0.1524" layer="91"/>
 <label x="416.56" y="497.84" size="1.778" layer="95"/>
-</segment>
-</net>
+<pinref part="U1" gate="D" pin="MII1_TXD1"/>
+</segment>
+</net>

Commit message: Add HDMI
Parts:
- added J1: 1-1747981-1, 1-1747981-1:1-1747981-1
Connections:
- net CEC: now also J1.7
- net DVI_5V: now also J1.2
- net GND: now also J1.12, J1.15, J1.18, J1.3, J1.6, J1.9
- net HDMI.DSCL: now also J1.5
- net HDMI.DSDA: now also J1.4
- net HPD: now also J1.1
- net TX0+: now also J1.13
- net TX0-: now also J1.11
- net TX1+: now also J1.16
- net TX1-: now also J1.14
- net TX2+: now also J1.19
- net TX2-: now also J1.17
- net TXC+: now also J1.10
- net TXC-: now also J1.8

Commit message: USR LED connections
Connections:
- net I2C0_SCL: now also U1A.I2C0_SCL, U1A.PMIC_SCL
- net I2C0_SDA: now also U1A.I2C0_SDA, U1A.PMIC_SDA
- net PWR_BUT: now also U1A.PMIC_PB_IN
- net USB_DC: now also U1A.VIN_USB@2, U1A.VIN_USB@3
- net USR0: now also U1C.GPMC_A5
- net USR1: now also U1C.GPMC_A6
- net USR2: now also U1C.GPMC_A7
- net USR3: now also U1C.GPMC_A8
Other:
- moved on the sheet: C48, C49, FB5, FB6, IC13, IC17, IC4, POWER, PWR, R123, R17, R24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

Commit message: Power and other clean-up
Parts:
- removed C18: .1uF, 6.3V, rcl:C-USC0402K
- removed R40: 10k, 1%, rcl:R-US_R0402
- removed R41, R42: 1.5k, 1%, rcl:R-US_R0402
- removed R54: 0, 1%, rcl:R-US_R0402
- added BT1: LTST-C191TBKT, GHI-BasicComponents:LED-(INCH)-0603
- added R9: 1k, rcl:R-US_R0402
- added T1: BSS138W-7-F, GHI Transistors:BSS138W-7-F
Connections:
- removed net GPIO1_16: R54.1
- removed net GPIO1_16.SIP: R54.2
- removed net GPIO3_21: R110.2
- removed net HDMICLK_DIS#: OSC1.INH#
- removed net N$54: R40.2, TP1.TP
- removed net SPI1_CS0: IC9.AP1
- removed net SPI1_D0: IC9.AP0
- removed net SPI1_SCLK: IC9.ACLK
- new net EEPROM_WP: TP1.TP, U1A.EEPROM_WP, U1C.GPMC_BEN0_CLE
- new net HDMI_AUDBCLK: IC9.ACLK, U1C.MCASP0_ACLKX
- new net HDMI_AUDCLK: R110.2, U1C.MCASP0_AHCLKX
- new net HDMI_AUDCLK_DIS#: OSC1.INH#, U1C.GPMC_A11
- new net HDMI_AUDDOUT: IC9.AP1, U1C.MCASP0_AHCLKR
- new net HDMI_AUDWCLK: IC9.AP0, U1C.MCASP0_FSX
- new net N$2: BT1.A, R9.1
- new net N$21: U1A.PMIC_POWER_EN, U1A.PMIC_PWR_EN
- new net N$23: U1A.PMIC_LDO_PGOOD, U1A.RTC_PWRONRSTN
- new net N$26: U1A.EXT_WAKEUP, U1A.PMIC_NWAKEUP
- new net N$27: U1A.EXTINTN, U1A.PMIC_NINT
- new net N$8: BT1.K, T1.D
- new net VDD_RTC: U1A.SYS_RTC_1P8V@2
- new net WIFI_LED(GPIO3_01): T1.G, U1D.MII1_CRS
- net 3.3V-WIFI: now also R9.2
- net GND: now also T1.S; no longer C18.2
- net HDMI_INT: now also U1C.GPMC_A9
- net I2C0_SCL: no longer R41.2
- net I2C0_SDA: no longer R42.2
- net SYS_5V: now also U1A.SYS_VOUT@3, U1A.SYS_VOUT@4
- net USB1_OC#: now also U1C.GPMC_A10
- net VDD_3V3AUX: now also U1A.SYS_VDD2_3P3V@2
- net VDD_3V3B: now also U1A.SYS_VDD1_3P3V@2, U1A.SYS_VDD1_3P3V@4; no longer C18.1, R40.1, R41.1, R42.1
Other:
- note removed: "EEPROM"
- moved on the sheet: C47, OSC1, POWER, R110, TP1

Commit message: Power and other clean-up
Parts:
- removed FB7: 1k BLM15AG102SN1D, rcl:R-US_R0402
- removed R14: 0, 1%, rcl:R-US_R0402
Connections:
- net CLKOUT2: no longer FB7.1, R14.1
- net N$28: now also U1B.SYS_ADC_1P8V, U1B.VREFP; no longer R14.2
- net N$29: now also U1B.AGND_ADC, U1B.VREFN; no longer FB7.2
- net PMIC_PGOOD: now also U1A.PMIC_PGOOD, U1A.PWRONRSTN
- net SYS_5V: now also U1A.SYS_VOUT@1, U1A.SYS_VOUT@2
- net SYS_RESET#: now also U1A.WARMRSTN
- net VDD_3V3AUX: now also U1A.SYS_VDD2_3P3V@1
- net VDD_3V3B: now also U1A.SYS_VDD1_3P3V@1, U1A.SYS_VDD1_3P3V@3
- net VDD_RTC: now also U1A.SYS_RTC_1P8V@1
Other:
- note removed: "RESET#"
- moved on the sheet: C16, IC2, R32, RESET

Commit message: Stopping for the night
Parts:
- added U2: A3967SLBTR, A3967SLBTR:A3967SLBTR
Connections:
- new net N$30: R9.2
- net 3.3V-WIFI: no longer R9.2
Other:
- note added: "Motor Driver"
- note removed: "Prototyped by: GHI Electronics, LLC"
Changed lines of the file:
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@@
 <part name="GND4" library="supply1" deviceset="GND" device=""/>
 <part name="T1" library="GHI Transistors" deviceset="BSS138W-7-F" device="" value="BSS138W-7-F"/>
-<part name="SUPPLY8" library="GHI-PowerGoundSupply" deviceset="3.3V-WIFI" device=""/>
+<part name="U2" library="A3967SLBTR" deviceset="A3967SLBTR" device=""/>
 </parts>
 <sheets>
@@
 <text x="58.42" y="571.5" size="12.7" layer="94" ratio="10">OSD3358 SiP</text>
 <text x="822.706" y="6.35" size="3.81" layer="94" font="vector">A0</text>
-<text x="751.84" y="38.1" size="2.1844" layer="94" font="vector">Prototyped by: GHI Electronics, LLC</text>
 <rectangle x1="755.533009375" y1="23.854834375" x2="756.376853125" y2="23.919746875" layer="200"/>
 <rectangle x1="758.648740625" y1="23.854834375" x2="759.427671875" y2="23.919746875" layer="200"/>
@@
 <rectangle x1="756.636496875" y1="34.759903125" x2="758.194365625" y2="34.824809375" layer="200"/>
 <rectangle x1="756.961053125" y1="34.8248125" x2="757.869809375" y2="34.889725" layer="200"/>
+<text x="480.06" y="91.44" size="6.4516" layer="94" ratio="10">Motor Driver</text>
 </plain>
 <instances>
@@
 <instance part="GND4" gate="1" x="274.32" y="205.74" rot="MR0"/>
 <instance part="T1" gate="G$1" x="274.32" y="215.9"/>
-<instance part="SUPPLY8" gate="G$1" x="274.32" y="248.92"/>
+<instance part="U2" gate="G$1" x="515.62" y="45.72"/>
 </instances>
 <busses>
@@
 <junction x="261.62" y="353.06"/>
 </segment>
-<segment>
-<pinref part="R9" gate="G$1" pin="2"/>
-<wire x1="274.32" y1="246.38" x2="274.32" y2="243.84" width="0.1524" layer="91"/>
-<pinref part="SUPPLY8" gate="G$1" pin="3.3V-WIFI"/>
-</segment>
 </net>
 <net name="1.8V-WIFI" class="0">
@@
 </segment>
 </net>
+<net name="N$30" class="0">
+<segment>
+<pinref part="R9" gate="G$1" pin="2"/>
+<wire x1="274.32" y1="246.38" x2="274.32" y2="243.84" width="0.1524" layer="91"/>
+</segment>
+</net>

Commit message: Started motor driver
Parts:
- added C12: 1uF,10V, Seeed-Capacitor:CERAMIC-1UF-10V-10%-X5R(0402)
- added C7: 47uF,50V, resistor:CPOL-USF
- added C9: 100nF,50V, Seeed-Capacitor:CERAMIC-100NF-50V-10%-X7R(0805)
- added R12: 10K, Seeed-Resistor:DIP-VR-TOP-ADJ-10K(3P-9.5X9.5X5MM)
- added R13: 2K, Seeed-Resistor:SMD-RES-2K-1%-1/10W(0603)
Connections:
- new net 12VDC: C7.+, IC4.VI, X12.IN
- new net N$31: R12.1, R13.2
- net GND: now also C7.-, R13.1
- net N$10: now also R12.3, U2.REF; no longer IC4.VI, X12.IN
- net VDD_5V: now also R12.2, U2.VCC
Other:
- moved on the sheet: X12
Changed lines of the file:
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@@
 <setting verticaltext="up"/>
 </settings>
-<grid distance="0.1" unitdist="inch" unit="inch" style="lines" multiple="1" display="no" altdistance="0.01" altunitdist="inch" altunit="inch"/>
+<grid distance="0.05" unitdist="inch" unit="inch" style="lines" multiple="1" display="no" altdistance="0.01" altunitdist="inch" altunit="inch"/>
 <layers>
 <layer number="1" name="Top" color="4" fill="1" visible="no" active="no"/>
@@
 <layer number="136" name="silktop" color="7" fill="1" visible="yes" active="yes"/>
 <layer number="137" name="silkbottom" color="7" fill="1" visible="yes" active="yes"/>
+<layer number="138" name="mbTest" color="7" fill="1" visible="yes" active="yes"/>
+<layer number="139" name="mtKeepout" color="7" fill="1" visible="yes" active="yes"/>
+<layer number="140" name="mbKeepout" color="7" fill="1" visible="yes" active="yes"/>
+<layer number="141" name="mtRestrict" color="7" fill="1" visible="yes" active="yes"/>
+<layer number="142" name="mbRestrict" color="7" fill="1" visible="yes" active="yes"/>
+<layer number="143" name="mvRestrict" color="7" fill="1" visible="yes" active="yes"/>
 <layer number="144" name="Drill_legend" color="7" fill="1" visible="yes" active="yes"/>
 <layer number="145" name="DrillLegend_01-16" color="7" fill="1" visible="yes" active="yes"/>
 <layer number="146" name="DrillLegend_01-20" color="7" fill="1" visible="yes" active="yes"/>
+<layer number="147" name="mMeasures" color="7" fill="1" visible="yes" active="yes"/>
+<layer number="148" name="mDocument" color="7" fill="1" visible="yes" active="yes"/>
+<layer number="149" name="mReference" color="7" fill="1" visible="yes" active="yes"/>
 <layer number="150" name="Notes" color="7" fill="1" visible="no" active="yes"/>
 <layer number="151" name="HeatSink" color="14" fill="1" visible="no" active="no"/>
@@
 <layer number="154" name="FabDoc2" color="2" fill="1" visible="no" active="no"/>
 <layer number="155" name="FabDoc3" color="7" fill="15" visible="no" active="no"/>
+<layer number="166" name="AntennaArea" color="7" fill="1" visible="yes" active="yes"/>
+<layer number="168" name="4mmHeightArea" color="7" fill="1" visible="yes" active="yes"/>
+<layer number="191" name="mNets" color="7" fill="1" visible="yes" active="yes"/>
+<layer number="192" name="mBusses" color="7" fill="1" visible="yes" active="yes"/>
+<layer number="193" name="mPins" color="7" fill="1" visible="yes" active="yes"/>
+<layer number="194" name="mSymbols" color="7" fill="1" visible="yes" active="yes"/>
+<layer number="195" name="mNames" color="7" fill="1" visible="yes" active="yes"/>
+<layer number="196" name="mValues" color="7" fill="1" visible="yes" active="yes"/>
 <layer number="199" name="Contour" color="7" fill="1" visible="no" active="no"/>
 <layer number="200" name="200bmp" color="1" fill="10" visible="yes" active="yes"/>
@@
 <part name="T1" library="GHI Transistors" deviceset="BSS138W-7-F" device="" value="BSS138W-7-F"/>
 <part name="U2" library="A3967SLBTR" deviceset="A3967SLBTR" device=""/>
+<part name="C7" library="resistor" library_urn="urn:adsk.eagle:library:348" deviceset="CPOL-US" device="F" package3d_urn="urn:adsk.eagle:package:25916/1" value="47uF,50V"/>
+<part name="C9" library="Seeed-Capacitor" deviceset="CERAMIC-100NF-50V-10%-X7R(0805)" device="" value="100nF,50V"/>
+<part name="C12" library="Seeed-Capacitor" deviceset="CERAMIC-1UF-10V-10%-X5R(0402)" device="" value="1uF,10V"/>
+<part name="SUPPLY8" library="GHI-PowerGoundSupply" deviceset="VDD_5V" device=""/>
+<part name="R12" library="Seeed-Resistor" deviceset="DIP-VR-TOP-ADJ-10K(3P-9.5X9.5X5MM)" device="" value="10K"/>
+<part name="R13" library="Seeed-Resistor" deviceset="SMD-RES-2K-1%-1/10W(0603)" device="" value="2K"/>
+<part name="GND11" library="supply1" deviceset="GND" device=""/>
 </parts>
 <sheets>
@@
 </instance>
 <instance part="R56" gate="G$1" x="43.18" y="502.92" rot="R90"/>
-<instance part="X12" gate="G$1" x="660.4" y="566.42"/>
+<instance part="X12" gate="G$1" x="632.46" y="566.42"/>
 <instance part="U1" gate="A" x="711.2" y="398.78"/>
 <instance part="U1" gate="B" x="68.58" y="436.88"/>
@@
 <instance part="T1" gate="G$1" x="274.32" y="215.9"/>
 <instance part="U2" gate="G$1" x="515.62" y="45.72"/>
+<instance part="C7" gate="G$1" x="650.24" y="571.5"/>
+<instance part="C9" gate="G$1" x="665.48" y="571.5" rot="R90"/>
+<instance part="C12" gate="G$1" x="685.8" y="568.96"/>
+<instance part="SUPPLY8" gate="G$1" x="459.74" y="76.2"/>
+<instance part="R12" gate="G$1" x="459.74" y="63.5" rot="R90"/>
+<instance part="R13" gate="G$1" x="459.74" y="52.07" rot="R90"/>
+<instance part="GND11" gate="1" x="459.74" y="43.18"/>
 </instances>
 <busses>
@@
 <wire x1="668.02" y1="561.34" x2="665.48" y2="561.34" width="0.1524" layer="91"/>
 <pinref part="IC4" gate="A1" pin="GND"/>
+<wire x1="665.48" y1="561.34" x2="650.24" y2="561.34" width="0.1524" layer="91"/>
+<wire x1="650.24" y1="561.34" x2="637.54" y2="561.34" width="0.1524" layer="91"/>
 <wire x1="678.18" y1="571.5" x2="678.18" y2="568.96" width="0.1524" layer="91"/>
 <wire x1="678.18" y1="568.96" x2="670.56" y2="568.96" width="0.1524" layer="91"/>
@@
 <wire x1="670.56" y1="563.88" x2="668.02" y2="563.88" width="0.1524" layer="91"/>
 <wire x1="668.02" y1="563.88" x2="668.02" y2="561.34" width="0.1524" layer="91"/>
+<pinref part="C7" gate="G$1" pin="-"/>
+<wire x1="650.24" y1="566.42" x2="650.24" y2="561.34" width="0.1524" layer="91"/>
+<wire x1="665.48" y1="568.96" x2="665.48" y2="561.34" width="0.1524" layer="91"/>
+<junction x="665.48" y="561.34"/>
+<junction x="650.24" y="561.34"/>
+<wire x1="678.18" y1="568.96" x2="683.26" y2="568.96" width="0.1524" layer="91"/>
+<junction x="678.18" y="568.96"/>
 </segment>
 <segment>
@@
 <wire x1="274.32" y1="208.28" x2="274.32" y2="210.82" width="0.1524" layer="91"/>
 </segment>
+<segment>
+<pinref part="GND11" gate="1" pin="GND"/>
+<pinref part="R13" gate="G$1" pin="1"/>
+<wire x1="459.74" y1="45.72" x2="459.74" y2="48.26" width="0.1524" layer="91"/>
+</segment>
 </net>
 <net name="N$6" class="0">
@@
 <pinref part="IC4" gate="A1" pin="VO"/>
 <wire x1="688.34" y1="579.12" x2="693.42" y2="579.12" width="0.1524" layer="91"/>
-<wire x1="693.42" y1="579.12" x2="693.42" y2="566.42" width="0.1524" layer="91"/>
+<wire x1="693.42" y1="579.12" x2="693.42" y2="568.96" width="0.1524" layer="91"/>
+<wire x1="693.42" y1="568.96" x2="693.42" y2="566.42" width="0.1524" layer="91"/>
 <wire x1="693.42" y1="566.42" x2="701.04" y2="566.42" width="0.1524" layer="91"/>
 <pinref part="U1" gate="A" pin="VIN_AC@1"/>
@@
 <wire x1="701.04" y1="561.34" x2="701.04" y2="563.88" width="0.1524" layer="91"/>
 <junction x="701.04" y="563.88"/>
+<wire x1="688.34" y1="568.96" x2="693.42" y2="568.96" width="0.1524" layer="91"/>
+<junction x="693.42" y="568.96"/>
 </segment>
 <segment>
@@
 <wire x1="86.36" y1="386.08" x2="88.9" y2="386.08" width="0.1524" layer="91"/>
 </segment>
+<segment>
+<pinref part="U2" gate="G$1" pin="VCC"/>
+<pinref part="SUPPLY8" gate="G$1" pin="VDD_5V"/>
+<wire x1="497.84" y1="71.12" x2="459.74" y2="71.12" width="0.1524" layer="91"/>
+<wire x1="459.74" y1="71.12" x2="459.74" y2="73.66" width="0.1524" layer="91"/>
+<pinref part="R12" gate="G$1" pin="2"/>
+<wire x1="459.74" y1="68.58" x2="459.74" y2="71.12" width="0.1524" layer="91"/>
+<junction x="459.74" y="71.12"/>
+</segment>
 </net>
 <net name="PWR_BUT" class="0">
@@
 </segment>
 </net>
-<net name="N$10" class="0">
+<net name="12VDC" class="0">
 <segment>
 <pinref part="X12" gate="G$1" pin="IN"/>
-<wire x1="665.48" y1="566.42" x2="668.02" y2="566.42" width="0.1524" layer="91"/>
+<wire x1="637.54" y1="566.42" x2="642.62" y2="566.42" width="0.1524" layer="91"/>
 <pinref part="IC4" gate="A1" pin="VI"/>
-<wire x1="668.02" y1="566.42" x2="668.02" y2="579.12" width="0.1524" layer="91"/>
+<wire x1="642.62" y1="566.42" x2="642.62" y2="579.12" width="0.1524" layer="91"/>
+<wire x1="642.62" y1="579.12" x2="650.24" y2="579.12" width="0.1524" layer="91"/>
+<pinref part="C7" gate="G$1" pin="+"/>
+<wire x1="650.24" y1="579.12" x2="665.48" y2="579.12" width="0.1524" layer="91"/>
+<wire x1="665.48" y1="579.12" x2="668.02" y2="579.12" width="0.1524" layer="91"/>
+<wire x1="650.24" y1="574.04" x2="650.24" y2="579.12" width="0.1524" layer="91"/>
+<wire x1="665.48" y1="574.04" x2="665.48" y2="579.12" width="0.1524" layer="91"/>
+<junction x="650.24" y="579.12"/>
+<junction x="665.48" y="579.12"/>
+<label x="642.62" y="579.12" size="1.778" layer="95"/>
 </segment>
 </net>
@@
 </segment>
 </net>
+<net name="N$10" class="0">
+<segment>
+<pinref part="R12" gate="G$1" pin="3"/>
+<wire x1="464.82" y1="63.5" x2="472.44" y2="63.5" width="0.1524" layer="91"/>
+<wire x1="472.44" y1="63.5" x2="472.44" y2="66.04" width="0.1524" layer="91"/>
+<pinref part="U2" gate="G$1" pin="REF"/>
+<wire x1="472.44" y1="66.04" x2="497.84" y2="66.04" width="0.1524" layer="91"/>
+</segment>
+</net>
+<net name="N$31" class="0">
+<segment>
+<pinref part="R12" gate="G$1" pin="1"/>
+<wire x1="459.74" y1="55.88" x2="459.74" y2="58.42" width="0.1524" layer="91"/>
+<pinref part="R13" gate="G$1" pin="2"/>
+</segment>
+</net>
