File: EAGLE/whitherbone.sch (EAGLE design)
At the start: 220 parts, among them IC1 A4983, IC12 TPS2051BDGN, IC13 SN74AUC1G74, IC14 TPD4S012DRY, IC15 TPD4S012DRY, IC17 SN74LVC2G241DCUR, IC2 SN74LVC1G07DCK, IC4 7805T, IC7 IP4283CZ10-TBR, IC8 IP4283CZ10-TBR, IC9 TDA19988BHN/C1,557, J1 1-1747981-1, Q2 32.768kHz, Q4 24 MHz, T1 BSS138W-7-F, T3 BSS138W-7-F, T4 BSS138W-7-F, U1 OSD3358-512M-BSM, U2 SN74AHCT125PW, X2 SCHA5B0200, X4 10118192-0001LF

Commit message: Add quick fan connector
Parts:
- added C21: 1uF,10V, Seeed-Capacitor:CERAMIC-1UF-10V-10%-X5R(0402)
- added JP2: (no value), SparkFun:M04PTH
Connections:
- net GND: now also JP1.4, JP2.1, JP2.4
- net VDD_5V: now also JP1.2, JP2.2, JP2.3; no longer JP1.4
Other:
- note added: "FAN Connector"
Changed lines of the file:
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@@
 <part name="U2" library="SN74AHCT125PW" deviceset="SN74AHCT125PW" device=""/>
 <part name="C19" library="Seeed-Capacitor" deviceset="CERAMIC-1UF-10V-10%-X5R(0402)" device="" value="1uF,10V"/>
+<part name="JP2" library="SparkFun" deviceset="M04" device="PTH"/>
+<part name="GND28" library="supply1" deviceset="GND" device=""/>
+<part name="SUPPLY18" library="GHI-PowerGoundSupply" deviceset="VDD_5V" device=""/>
+<part name="C21" library="Seeed-Capacitor" deviceset="CERAMIC-1UF-10V-10%-X5R(0402)" device="" value="1uF,10V"/>
 </parts>
 <sheets>
@@
 <text x="548.386" y="20.32" size="1.778" layer="98">Motor current 0mA to over 2A/phase</text>
 <text x="652.78" y="144.78" size="6.4516" layer="94" ratio="10">Neopixel Connector</text>
+<text x="228.6" y="678.18" size="6.4516" layer="94" ratio="10">FAN Connector</text>
 </plain>
 <instances>
@@
 <instance part="GND26" gate="1" x="172.72" y="492.76" rot="R90"/>
 <instance part="JP1" gate="G$1" x="734.06" y="119.38" rot="MR0"/>
-<instance part="GND27" gate="1" x="716.28" y="111.76" rot="MR0"/>
+<instance part="GND27" gate="1" x="718.82" y="111.76" rot="MR0"/>
 <instance part="SUPPLY10" gate="G$1" x="716.28" y="129.54" rot="MR0"/>
 <instance part="U2" gate="A" x="683.26" y="109.22"/>
 <instance part="C19" gate="G$1" x="706.12" y="111.76" rot="R90"/>
+<instance part="JP2" gate="G$1" x="264.16" y="655.32" rot="MR0"/>
+<instance part="GND28" gate="1" x="248.92" y="647.7" rot="MR0"/>
+<instance part="SUPPLY18" gate="G$1" x="246.38" y="665.48" rot="MR0"/>
+<instance part="C21" gate="G$1" x="236.22" y="647.7" rot="R90"/>
 </instances>
 <busses>
@@
 <segment>
 <pinref part="JP1" gate="G$1" pin="1"/>
-<wire x1="728.98" y1="116.84" x2="716.28" y2="116.84" width="0.1524" layer="91"/>
+<wire x1="728.98" y1="116.84" x2="718.82" y2="116.84" width="0.1524" layer="91"/>
 <label x="726.44" y="116.84" size="1.778" layer="95" rot="MR0"/>
 <pinref part="GND27" gate="1" pin="GND"/>
-<wire x1="716.28" y1="116.84" x2="716.28" y2="114.3" width="0.1524" layer="91"/>
-<wire x1="716.28" y1="116.84" x2="711.2" y2="116.84" width="0.1524" layer="91"/>
-<junction x="716.28" y="116.84"/>
+<wire x1="718.82" y1="116.84" x2="718.82" y2="114.3" width="0.1524" layer="91"/>
+<wire x1="718.82" y1="116.84" x2="711.2" y2="116.84" width="0.1524" layer="91"/>
+<junction x="718.82" y="116.84"/>
 <pinref part="U2" gate="A" pin="GND"/>
 <wire x1="665.48" y1="91.44" x2="662.94" y2="91.44" width="0.1524" layer="91"/>
@@
 <wire x1="706.12" y1="104.14" x2="706.12" y2="109.22" width="0.1524" layer="91"/>
 <junction x="711.2" y="104.14"/>
+<wire x1="718.82" y1="116.84" x2="718.82" y2="124.46" width="0.1524" layer="91"/>
+<pinref part="JP1" gate="G$1" pin="4"/>
+<wire x1="718.82" y1="124.46" x2="728.98" y2="124.46" width="0.1524" layer="91"/>
+</segment>
+<segment>
+<pinref part="JP2" gate="G$1" pin="1"/>
+<wire x1="259.08" y1="652.78" x2="248.92" y2="652.78" width="0.1524" layer="91"/>
+<label x="256.54" y="652.78" size="1.778" layer="95" rot="MR0"/>
+<pinref part="GND28" gate="1" pin="GND"/>
+<wire x1="248.92" y1="652.78" x2="248.92" y2="650.24" width="0.1524" layer="91"/>
+<wire x1="248.92" y1="652.78" x2="241.3" y2="652.78" width="0.1524" layer="91"/>
+<junction x="248.92" y="652.78"/>
+<wire x1="241.3" y1="640.08" x2="241.3" y2="652.78" width="0.1524" layer="91"/>
+<wire x1="236.22" y1="640.08" x2="241.3" y2="640.08" width="0.1524" layer="91"/>
+<wire x1="236.22" y1="640.08" x2="236.22" y2="645.16" width="0.1524" layer="91"/>
+<wire x1="248.92" y1="652.78" x2="248.92" y2="660.4" width="0.1524" layer="91"/>
+<pinref part="JP2" gate="G$1" pin="4"/>
+<wire x1="248.92" y1="660.4" x2="259.08" y2="660.4" width="0.1524" layer="91"/>
 </segment>
 </net>
@@
 </segment>
 <segment>
-<wire x1="716.28" y1="124.46" x2="716.28" y2="127" width="0.1524" layer="91"/>
+<wire x1="716.28" y1="119.38" x2="716.28" y2="127" width="0.1524" layer="91"/>
 <pinref part="SUPPLY10" gate="G$1" pin="VDD_5V"/>
-<wire x1="706.12" y1="137.16" x2="706.12" y2="124.46" width="0.1524" layer="91"/>
-<wire x1="706.12" y1="124.46" x2="716.28" y2="124.46" width="0.1524" layer="91"/>
-<pinref part="JP1" gate="G$1" pin="4"/>
-<wire x1="716.28" y1="124.46" x2="728.98" y2="124.46" width="0.1524" layer="91"/>
+<wire x1="706.12" y1="137.16" x2="706.12" y2="119.38" width="0.1524" layer="91"/>
+<wire x1="706.12" y1="119.38" x2="716.28" y2="119.38" width="0.1524" layer="91"/>
 <pinref part="U2" gate="A" pin="VCC"/>
 <wire x1="665.48" y1="121.92" x2="660.4" y2="121.92" width="0.1524" layer="91"/>
@@
 <junction x="660.4" y="111.76"/>
 <junction x="660.4" y="121.92"/>
-<junction x="716.28" y="124.46"/>
-<wire x1="706.12" y1="124.46" x2="706.12" y2="114.3" width="0.1524" layer="91"/>
-<junction x="706.12" y="124.46"/>
+<wire x1="706.12" y1="119.38" x2="706.12" y2="114.3" width="0.1524" layer="91"/>
+<junction x="706.12" y="119.38"/>
+<pinref part="JP1" gate="G$1" pin="2"/>
+<wire x1="716.28" y1="119.38" x2="728.98" y2="119.38" width="0.1524" layer="91"/>
+<junction x="716.28" y="119.38"/>
+</segment>
+<segment>
+<wire x1="246.38" y1="657.86" x2="246.38" y2="662.94" width="0.1524" layer="91"/>
+<pinref part="SUPPLY18" gate="G$1" pin="VDD_5V"/>
+<wire x1="236.22" y1="657.86" x2="246.38" y2="657.86" width="0.1524" layer="91"/>
+<wire x1="236.22" y1="657.86" x2="236.22" y2="650.24" width="0.1524" layer="91"/>
+<pinref part="JP2" gate="G$1" pin="2"/>
+<wire x1="246.38" y1="657.86" x2="246.38" y2="655.32" width="0.1524" layer="91"/>
+<wire x1="246.38" y1="655.32" x2="259.08" y2="655.32" width="0.1524" layer="91"/>
+<pinref part="JP2" gate="G$1" pin="3"/>
+<wire x1="246.38" y1="657.86" x2="259.08" y2="657.86" width="0.1524" layer="91"/>
+<junction x="246.38" y="657.86"/>
 </segment>
 </net>

Commit message: Use version from Seeed
Parts:
- removed ANT1, ANT2: U.FL-R-SMT-1(10), GHI-Connectors:U.FL-R-SMT-1
- removed BT, BT1, PWR, USR0, USR1, USR2, USR3, WL: LTST-C191TBKT, GHI-BasicComponents:LED-(INCH)-0603
- removed FB4: 0.1 Ohm, 0805, GHI-BasicComponents:FB-(INCH)-0805
- removed IC13: SN74AUC1G74, GHI-IC:SN74AUC1G74
- removed IC14: TPD4S012DRY, GHI-IC:TPD4S012DRYR
- removed IC17: SN74LVC2G241DCUR, GHI-IC:SN74LVC2G241DCUR
- removed IC2: SN74LVC1G07DCK, GHI-IC:SN74LVC1G07DCK
- removed IC4: 7805T, linear:7805T
- removed IC7, IC8: IP4283CZ10-TBR, GHI-IC:IP4283CZ10IP4283CZ10-TBR
- removed IC9: TDA19988BHN/C1,557, GHI-IC:TDA19988BHN/C1
- removed OSC1: ASDMB-24.576MHZ-LC-T, GHI2:OSC-2.5X2.0
- removed OSC2: NZ2520SB-32.768KHZ-NSA3534C, GHI-IC:OSCILLATOR
- removed POWER, RESET: MINI_PUSHBUTTON, GHI2:MINI_PUSHBUTTON
- removed Q2: 32.768kHz, GHI2:CRYSTAL_3.2X1.5
- removed Q4: 24 MHz, GHI2:CRYSTAL_5X3.2MM
- removed R101: 10k, rcl:R-US_R0402
- removed R115, R118: 1.5k, 1%, rcl:R-US_R0402
- removed R119, R121: 10k, 1%, rcl:R-US_R0402
- removed R120: 27k, 1%, rcl:R-US_R0402
- removed R123, R76: 100k, 1%, rcl:R-US_R0402
- removed R23: 20K, SparkFun:RESISTOR0402-RES
- removed X1: (no value), GHI-Headers:1X6-(INCH)-0.1-TH
- removed X12: (no value), GHI-Connectors:PJ-102B_POWER_CON
- removed X3: (no value), GHI2:USB_HOST_W/CHASSIS_GND
- removed X4: 10118192-0001LF, GHI-Connectors:10118192-0001LF
- added ANT3, ANT4: (no value), Connector-new:ANTENNA-U-FL-2.6X2.6
- added C22: 0.1uF, 6.3V, Discrete-new:CAP-0402
- added C25, C26: 47pF, Discrete-new:CAP-0402
- added C45, C65, C69, C76: 100nF, Discrete-new:CAP-0402
- added C66: .1uF, 6.3V, Discrete-new:CAP-0402
- added C67: 22nF, Discrete-new:CAP-0402
- added C68: 100nF, Discrete-new:CAP-0603
- added C70, C71: 47uF 25V, Discrete-new:CAP-POLAR-ELECTRO-C
- added C72: 220nF, Discrete-new:CAP-0402
- added C73: 100nF, Discrete-new:CAP-0805
- added C74: DNI, Discrete-new:CAP-0402
- added C75: 1uF 10V, Discrete-new:CAP-0402
- added C77, C78, C80, C82, C83, C84: 10uF, Discrete-new:CAP-0805
- added C79: 22uF, Discrete-new:CAP-POLAR-ELECTRO-B
- added C81: 22uF 16V, Discrete-new:CAP-1206
- added D10, D12, D13, D2, D3: DF2S6.8FS, Discrete-new:D-ESD-2P'DF2S6.8FS'
- added D11, D4, D5, D6, D7, D8, D9: (no value), Discrete-new:LED'0603'
- added J2: (no value), Connector-new:HEADER-2P-65/35MIL
- added J3: 6p-2.54, OSD3358-SM-RED Platform:826646-6
- added J4: ST-HD-010, template:CONNECTOR-HDMI-19P
- added J5: (no value), Connector-new:MICRO-SD-CARD-HOLDER-9P'MICROSD-9P'
- added J6: DC Power Jack, For_Test_Albert:DC-044
- added J7: (no value), Connector-new:SCREW-TERMINAL-4P'3.5'
- added J8: (no value), Connector-new:MICRO-USB5+4P-320010050
- added L1, L4: WPN201610MR47MT, Discrete-new:L-MPM201610SR33_T
- added L2: 10uH, Discrete-new:INDUCTOR/FERRITE-BEAD5040S
- added Q1: MMBT2907, Discrete-new:TRANSISTOR-PNP
- added R106, R107, R108, R109, R112, R113: 33R, Discrete-new:RES-0402
- added R30, R51: 0R, Discrete-new:RES-0402
- added R31, R44: 22R, Discrete-new:RES-0402
- added R33: 0, 1%, Discrete-new:RES-0402
- added R33333, R48, R74, R77, R79, R97: 10k, Discrete-new:RES-0402
- added R36, R38: 1.5K, 1%, Discrete-new:RES-0402
- added R40: 5.6K 1%, Discrete-new:RES-0402
- added R41, R42: 100k 1%, Discrete-new:RES-0402
- added R45, R46: 2k, Discrete-new:RES-0402
- added R47: 33k, Discrete-new:RES-0402
- added R49, R50: 10K, Discrete-new:RES-0402
- added R54: 10k, 1%, Discrete-new:RES-0402
- added R59, R81, R82, R83: 100K, 1%, Discrete-new:RES-0402
- added R84: 3.3k, Discrete-new:RES-0402
- added R86, R89, R91: 10K, 1%, Discrete-new:RES-0402
- added R93: 510R 1%, Discrete-new:RES-0402
- added R94: 24k, Discrete-new:RES-0402
- added SW1, SW2: (no value), Discrete-new:BUTTON-4P+
- added TP11, TP21, TP22, TP23, TP24, TP3, TP4: TPB0,65, OSD3358-SM-RED Platform:TPB0,65
- added TP20, TP25, TP27, TP28, TP29, TP30, TP31, TP32, TP9: (no value), Discrete-new:TEST-POINT'4545'
- added TP26, TP5, TP6, TP7, TP8: TESTPAD/W_HOLE_1X1, OSD3358-SM-RED Platform:TESTPAD/W_HOLE_1X1
- added TP33: TPPAD1-13, testpad:TPPAD1-13
- added U10: (no value), IC-new:LOGIC-SN74AUP1G125'DCK'
- added U11, U9: ESD-RCLAMP0524P, Discrete-new:ESD-RCLAMP0524P
- added U12: TL431, IC-new:PMIC-CJ432'CJ432'
- added U13: (no value), IC-new:LOGIC-SN74LVC1G07-DCK
- added U3: MP1496DJ-LF-2, IC-new:CONVERTER-MP1496DJ
- added U4: APX811, IC-new:SUPERVISOR-APX811-31UGSOT
- added U5, U8: ETA3410, IC-new:CONVERTER-ETA3410
- added U6: SN74LVC2G241_DCU_8, OSD3358-SM-RED Platform:SN74LVC2G241_DCU_8
- added U7: IT66121FN, IC-new:TRANSFER_IT66121FN-9
- added VIN: (no value), discrete:PAD-TEST-POINT'4545'
- added VR1: EVM3GSX50B14, Discrete-new:RES-ADJ-SMD
- added Y1: ABS07-32.768KHZ-T, OSD3358-SM-RED Platform:ABS07-32.768KHZ-T
- added Y2: 7A-24.000MAAJ-T, OSD3358-SM-RED Platform:7A-24.000MAAJ-T
- C1: value 10uF,10V -> 10uF; device rcl:C-USC0603K -> Discrete-new:CAP-0805
- C10: value .1uf -> 0.1uF, 6.3V; device SparkFun:CAP0402-CAP -> Discrete-new:CAP-0402
- C11: value 47uF DNP -> TLJB227M006R0500; device rcl:CPOL-USCT3528 -> Discrete-new:CAP-POLAR-AVX-B
- C12: value 1uF,10V -> 18pF, 50V; device Seeed-Capacitor:CERAMIC-1UF-10V-10%-X5R(0402) -> Discrete-new:CAP-0402
- C13, C14: value .1uf -> 100nF; device SparkFun:CAP0402-CAP -> Discrete-new:CAP-0402
- C15, C18: value .1uf -> 10uF; device SparkFun:CAP0402-CAP -> Discrete-new:CAP-0805
- C16: value 2.2uF, 6.3V -> 100nF; device rcl:C-USC0603K -> Discrete-new:CAP-0402
- C17: value .22uF -> 100nF; device SparkFun:CAP0402-CAP -> Discrete-new:CAP-0402
- C19: value 1uF,10V -> 10uF; device Seeed-Capacitor:CERAMIC-1UF-10V-10%-X5R(0402) -> Discrete-new:CAP-0805
- C2: value .1uF, 6.3V -> DNI; device rcl:C-USC0402K -> Discrete-new:CAP-0402
- C20: value 10uF, 6.3V -> 10uF; device rcl:C-USC0603K -> Discrete-new:CAP-0805
- C21: value 1uF,10V -> 10uF, 10V; device Seeed-Capacitor:CERAMIC-1UF-10V-10%-X5R(0402) -> Discrete-new:CAP-0805
- C23: value 47uF DNP -> 47pF; device rcl:CPOL-USCT3528 -> Discrete-new:CAP-0402
- C24: value .1uF, 6.3V -> 47pF; device rcl:C-USC0402K -> Discrete-new:CAP-0402
- C27, C28, C29, C30, C31, C32, C33, C34, C35, C36, C37, C38: value 47pF, 6.3V -> 47pF; device rcl:C-USC0402K -> Discrete-new:CAP-0402
- C3, C6: value 18pF, 50V -> 0.1uF, 6.3V; device rcl:C-USC0402K -> Discrete-new:CAP-0402
- C39, C40, C41: value 47pF, 6.3V -> 10uF; device rcl:C-USC0402K -> Discrete-new:CAP-0805
- C4, C5: device rcl:C-USC0402K -> Discrete-new:CAP-0402
- C42: value 47pF, 6.3V -> 1uF; device rcl:C-USC0402K -> Discrete-new:CAP-0402
- C43, C44, C47, C48, C49, C50, C51, C63: value .1uF, 6.3V -> 100nF; device rcl:C-USC0402K -> Discrete-new:CAP-0402
- C46, C60: value 10pF -> 100nF; device rcl:C-USC0402K -> Discrete-new:CAP-0402
- C52, C53: value .1uF, 6.3V -> 47uF DNP; device rcl:C-USC0402K -> Discrete-new:CAP-1206
- C54: value 2.2uF, 6.3V -> 220uF; device rcl:C-USC0603K -> Discrete-new:CAP-POLAR-AVX-E
- C55, C56: value 2.2uF, 6.3V -> 10pF; device rcl:C-USC0603K -> Discrete-new:CAP-0402
- C57: value 2.2uF, 6.3V -> 10uF; device rcl:C-USC0603K -> Discrete-new:CAP-0805
- C58: value .1uF, 6.3V -> 1uF; device rcl:C-USC0402K -> Discrete-new:CAP-0402
- C59: value .1uF, 6.3V -> DNP; device rcl:C-USC0402K -> Discrete-new:CAP-0402
- C61: value 10uF, 6.3V -> 100nF; device rcl:C-USC0603K -> Discrete-new:CAP-0402
- C62: value 220uF 6.3V -> 1uF; device rcl:CPOL-USD/7343-31W -> Discrete-new:CAP-0603
- C64: value 1uF, 6.3V -> 1uF; device rcl:C-USC0402K -> Discrete-new:CAP-0402
- C7: value 47uF,50V -> 18pF, 50V; device resistor:CPOL-USF -> Discrete-new:CAP-0402
- C8: value 1uF -> 1nF; device rcl:C-USC0402K -> Discrete-new:CAP-0402
- C9: value 100nF,50V -> 0.1uF, 6.3V; device Seeed-Capacitor:CERAMIC-100NF-50V-10%-X7R(0805) -> Discrete-new:CAP-0402
- D1: value RB751V40,115 -> (none); device GHI-BasicComponents:DIODE-SCHOTTKY-(NXP)-SOD323-(REFLOW) -> Discrete-new:LED'0603'
- F1: value 1206L025YR -> 100mA MF-FSMF010X; device inductor-neosid:SM-1206 -> Discrete-new:FUSE0603
- FB1, FB6, FB7, FB8: value 1k BLM15AG102SN1D -> BLM15PD121SN1D; device rcl:R-US_R0402 -> Discrete-new:INDUCTOR/FERRITE-BEAD'0402'
- FB2: value 2.5k Ohm (BLM18BD252SN1D) -> BLM15PD121SN1D; device GHI-BasicComponents:FB-(INCH)-0805 -> Discrete-new:INDUCTOR/FERRITE-BEAD'0402'
- FB3: device GHI-BasicComponents:FB-(INCH)-0805 -> Discrete-new:INDUCTOR/FERRITE-BEAD'0805'
- FB5: value 1k BLM15AG102SN1D -> 0.1 Ohm, 0805; device rcl:R-US_R0402 -> Discrete-new:INDUCTOR/FERRITE-BEAD'0805'
- FUD1, FUD2, FUD3, FUD4, FUD5, FUD6: device GHI:FIDUCIAL -> OSD3358-SM-RED Platform:FIDUCIAL
- IC1: device SparkFun:A4983 -> IC-new:TRANSLATOR-A4983
- IC12: device GHI-IC:TPS2051B -> IC-new:SWITCH-TPS2051B
- IC15: device GHI-IC:TPD4S012DRYR -> IC-new:TVS-TPD4S012DRYR
- J1: value 1-1747981-1 -> (none); device 1-1747981-1:1-1747981-1 -> Connector-new:HEADER-2P-65/35MIL
- MGT1, MGT2, MGT3, MGT4: device BeagleBoneBlack:MOUNTING_HOLE -> OSD3358-SM-RED Platform:MOUNTING_HOLE
- MOD1: device GHI-IC:WL1835MOD -> moudle-new:MODULE-RF-WL1835MOD
- R1: value 10k, 1% -> 10K, 1%; device rcl:R-US_R0402 -> Discrete-new:RES-0402
- R10: value .11 -> 0, 1%; device SparkFun:RESISTOR2010 -> Discrete-new:RES-0402
- R100, R104, R96: value 1k -> 10k; device rcl:R-US_R0402 -> Discrete-new:RES-0402
- R102, R103, R105, R111, R122, R124, R125: device rcl:R-US_R0402 -> Discrete-new:RES-0402
- R11: value 20K -> 0, 1%; device SparkFun:RESISTOR0402-RES -> Discrete-new:RES-0402
- R110: value 33 -> 33R; device rcl:R-US_R0402 -> Discrete-new:RES-0402
- R114: value 0, 1% -> 1k; device rcl:R-US_R0402 -> Discrete-new:RES-0402
- R12, R13: value 20K -> 1.5K, 1%; device SparkFun:RESISTOR0402-RES -> Discrete-new:RES-0402
- R14: value 20K -> 22k 1%; device SparkFun:RESISTOR0402-RES -> Discrete-new:RES-0402
- R140, R141, R142, R143: value 33, 5% -> 33R; device rcl:R-US_R0402 -> Discrete-new:RES-0402
- R15: value 20K -> 40.2K, 1%; device SparkFun:RESISTOR0402-RES -> Discrete-new:RES-0402
- R16: value 10K -> 0, 1%; device SparkFun:TRIMPOTSMD -> Discrete-new:RES-0402
- R17: value .1, 0805 -> DNP; device rcl:R-US_R0805 -> Discrete-new:RES-0402
- R18: value .11 -> 4.75K, 1%; device SparkFun:RESISTOR2010 -> Discrete-new:RES-0402
- R19: value 10k, 1% -> 10k; device rcl:R-US_R0402 -> Discrete-new:RES-0402
- R2, R3: value 10k, 1% -> 1k; device rcl:R-US_R0402 -> Discrete-new:RES-0402
- R20: value 20K -> 10K, 1%; device SparkFun:RESISTOR0402-RES -> Discrete-new:RES-0402
- R21: value 20K -> 499; device SparkFun:RESISTOR0402-RES -> Discrete-new:RES-0402
- R22: value 20K -> 4.75K, 1%; device SparkFun:RESISTOR0402-RES -> Discrete-new:RES-0402
- R24: value 10k, 1% -> 1M, 1%, DNI; device rcl:R-US_R0402 -> Discrete-new:RES-0402
- R25: value 2.49K -> 0, 1%; device SparkFun:RESISTOR0402-RES -> Discrete-new:RES-0402
- R26, R35, R37: value 0, 1% -> 1.5K, 1%; device rcl:R-US_R0402 -> Discrete-new:RES-0402
- R27: value 0, 1% -> 100K, 1%; device rcl:R-US_R0402 -> Discrete-new:RES-0402
- R28: value 47k, 1% -> 0R; device rcl:R-US_R0402 -> Discrete-new:RES-0402
- R29: value 22k, 1% -> 0R; device rcl:R-US_R0402 -> Discrete-new:RES-0402
- R32: value 10k, 1% -> 1M, 1%; device rcl:R-US_R0402 -> Discrete-new:RES-0402
- R34: value 22 -> 10k; device rcl:R-US_R0402 -> Discrete-new:RES-0402
- R39: value 0, 1% -> 10k; device rcl:R-US_R0402 -> Discrete-new:RES-0402
- R4: value 10k, 1% -> 22R; device rcl:R-US_R0402 -> Discrete-new:RES-0402
- R43: value 4.75k, 1% -> 22R; device rcl:R-US_R0402 -> Discrete-new:RES-0402
- R5: value 10k, 1% -> 0, 1%; device rcl:R-US_R0402 -> Discrete-new:RES-0402
- R52: value 4.75k, 1% -> DNP; device rcl:R-US_R0402 -> Discrete-new:RES-0402
- R53, R55: value 4.75k, 1% -> 100K, 1%; device rcl:R-US_R0402 -> Discrete-new:RES-0402
- R56: value DNP 1M, 1% -> 100K, 1%; device rcl:R-US_R0402 -> Discrete-new:RES-0402
- R57, R58, R61, R63, R67, R71: value 100k, 1% -> 100K, 1%; device rcl:R-US_R0402 -> Discrete-new:RES-0402
- R6: value 10k, 1% -> 100K, 1%, DNI; device rcl:R-US_R0402 -> Discrete-new:RES-0402
- R60, R62, R68: value 33, 5% -> 100K, 1%; device rcl:R-US_R0402 -> Discrete-new:RES-0402
- R64: value 33, 5% -> 100k; device rcl:R-US_R0402 -> Discrete-new:RES-0402
- R65: value 100k, 1% -> 0.1R; device rcl:R-US_R0402 -> Discrete-new:RES-1206
- R66: value 33, 5% -> 0.1R; device rcl:R-US_R0402 -> Discrete-new:RES-1206
- R69: value 100k, 1% -> 10R; device rcl:R-US_R0402 -> Discrete-new:RES-0402
- R7: value 10k, 1% -> 0R; device rcl:R-US_R0402 -> Discrete-new:RES-1206
- R70: value 33, 5% -> 10K; device rcl:R-US_R0402 -> Discrete-new:RES-0402
- R72: value 33, 5% -> 10k; device rcl:R-US_R0402 -> Discrete-new:RES-0402
- R73, R75, R78, R80: value 100k, 1% -> 10k; device rcl:R-US_R0402 -> Discrete-new:RES-0402
- R8: value 1M, 1% -> 1K, 1%; device rcl:R-US_R0402 -> Discrete-new:RES-0402
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Connections:
- net N$5 renamed AIN7
- removed net 12MHZ: FB6.2, IC9.OSC_IN/AP3
- removed net 12M_LOOP: IC13.D, IC13.Q#
- removed net 32.768KHZ: MOD1.EXT_32K, OSC2.OUT
- removed net DVI_5V: F1.1, J1.2, R115.1, R118.1
- removed net EXT_SWING: IC9.EXT_SWING, R119.1
- removed net HDMI.DSCL: IC9.DSCL, J1.5, R115.2
- removed net HDMI.DSDA: IC9.DSDA, J1.4, R118.2
- removed net HDMI_1V8: C50.1, C51.1, C52.1, C53.1, C54.1, C55.1, C56.1, C57.1, FB2.P$2, IC9.VDDA(1V8), IC9.VDDA1(PLL)(1V8), IC9.VDDA1(TX)(1V8)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
- removed net HDMI_AUDCLK: R110.2, U1C.MCASP0_AHCLKX
- removed net HDMI_AUDCLK_DIS#: OSC1.INH#, U1C.GPMC_A11
- removed net LCD.CLOCK: IC9.PCLK, R34.1
- removed net LCD.D0.B0--B3: C42.1, IC9.VPC[3], R87.2, U1D.LCD_DATA0
- removed net LCD.D1.B1--B4: C41.1, IC9.VPC[4], R85.2, U1D.LCD_DATA1
- removed net LCD.D10.G5--G7: C32.1, IC9.VPB[7], R67.2, U1D.LCD_DATA10
- removed net LCD.D11.R0--R3: C31.1, IC9.VPA[3], R65.2, U1D.LCD_DATA11
- removed net LCD.D12.R1--R4: C30.1, IC9.VPA[4], R63.2, U1D.LCD_DATA12
- removed net LCD.D13.R2--R5: C29.1, IC9.VPA[5], R61.2, U1D.LCD_DATA13
- removed net LCD.D14.R3--R6: C28.1, IC9.VPA[6], R58.1, U1D.LCD_DATA14
- removed net LCD.D15.R4--R7: C27.1, IC9.VPA[7], R57.2, U1D.LCD_DATA15
- removed net LCD.D2.B2--B5: C40.1, IC9.VPC[5], R88.1, U1D.LCD_DATA2
- removed net LCD.D3.B3--B6: C39.1, IC9.VPC[6], R80.1, U1D.LCD_DATA3
- removed net LCD.D4.B4--B7: C38.1, IC9.VPC[7], R78.1, U1D.LCD_DATA4
- removed net LCD.D5.G0--G2: C37.1, IC9.VPB[2], R76.1, U1D.LCD_DATA5
- removed net LCD.D6.G1--G3: C36.1, IC9.VPB[3], R75.2, U1D.LCD_DATA6
- removed net LCD.D7.G2--G4: C35.1, IC9.VPB[4], R73.2, U1D.LCD_DATA7
- removed net LCD.D8.G3--G5: C34.1, IC9.VPB[5], R71.2, U1D.LCD_DATA8
- removed net LCD.D9.G4--G6: C33.1, IC9.VPB[6], R69.2, U1D.LCD_DATA9
- removed net LCD.ENABLE: IC9.DE/FREF, R39.1
- removed net LCD.HSYNC: IC9.HSYNC/HREF, R37.1
- removed net LCD.VSYNC: IC9.VSYNC/VREF, R35.1
- removed net MCU.LCD.CLK: R34.2, U1D.LCD_PCLK
- removed net MCU.LCD.EN: R39.2, U1D.LCD_AC_BIAS_EN
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Other:
- note added: "1/12"
- note added: "12/12"
- note added: "2/12"
- note added: "3/12"
- note added: "32kHz Oscillator is used for RTC. If your application does not use the RTC, then this can be removed."
- note added: "4/12"
- note added: "5/12"
- note added: "9/12"
- note added: "AIN7 currently monitors the PMIC voltages via the internal PMIC mux. See the `Analog Multiplexer' section of the TPS65217 datasheet. For the internal PMIC voltages, there are dividers within the PMIC to keep the montiored voltages under 1.8V. However, PMIC_MUX_IN does not have any dividers and must be less than 1.8V. By default, PMIC_MUX_OUT is Hi-Z. The MUXCTRL register in the PMIC is used to se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"
- note added: "Battery Connector"
- note added: "Blue"
- note added: "Boot configuration"
- note added: "Clock resistors R32 and R24 may not be needed in your design. See https://octavosystems.com/osd335x/clock/ for more information."
- note added: "Clocks, Analog & USB"
- note added: "Configuration: - 24 MHz Crystal (SYSBOOT[14:15] = 01b) - CLKOUT1 disabled (SYSBOOT[5] = 0b)"
- note added: "Differential impedance: 100 Ohm"
- note added: "ESD Protection Diodes close to HDMI Connector."
- note added: "Fiducials"
- note added: "Green"
- note added: "HDMI"
- note added: "If the analog interface is not used, then VREFP and VREFN should be shorted to AGND."
- note added: "Maximum voltage for the analog inputs is 1.8V."
- note added: "Micro SD card slot"
- note added: "Mounting Holes"
- note added: "Mounting holes and other connector shields are part of a ground ring, CGND. This ring is connected to ground via a resistor on Page 1."
- note added: "PCADR pull high: 0x9A PCADR pull low : 0x98"
- note added: "Power & Reset"
- note added: "Power input protection. Adjust according to your application."
- note added: "RTC_KALDO_ENN is grounded thru a 10K ohm resistor so that the internal RTC LDO is enabled and CAP_VDD_RTC does not need to be connected to VDD_CORE."
- note added: "Red"
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
Commit message: Update to latest from Seeed
* Layout complete
* Added mechanical drawing (DXF) for board
Parts:
- removed FB1, FB6: BLM15PD121SN1D, Discrete-new:INDUCTOR/FERRITE-BEAD'0402'
- removed FB5: 0.1 Ohm, 0805, Discrete-new:INDUCTOR/FERRITE-BEAD'0805'
- removed IC12: TPS2051BDGN, IC-new:SWITCH-TPS2051B
- removed JP1, JP3: (no value), SparkFun:M04PTH
- removed JP5: (no value), BigEasyDriver_v11:M04SCREW_LOCK
- removed MOD1: WL1835MODGBMOCT, moudle-new:MODULE-RF-WL1835MOD
- removed R122: 0, 1%, Discrete-new:RES-0402
- removed R124, R125: 1k, Discrete-new:RES-0402
- removed R140, R141, R142, R143: 33R, Discrete-new:RES-0402
- removed R33333: 10k, Discrete-new:RES-0402
- removed T1, T3, T4: BSS138W-7-F, Discrete-new:MOSFET-N'SI1304BDL'
- removed TP33: TPPAD1-13, testpad:TPPAD1-13
- removed VIN: (no value), discrete:PAD-TEST-POINT'4545'
- removed X2: (no value), GHI2:USB_HOST_W/CHASSIS_GND
- removed Y2: 7A-24.000MAAJ-T, OSD3358-SM-RED Platform:7A-24.000MAAJ-T
- added L10: WPN201610MR47MT, Discrete-new:L-MPM201610SR33_T
- added L3: IHLP3232DZER100M01, Discrete-new:INDUCTOR/FERRITE-BEAD-IHLP3232DZER100M01
- added L6: LQH44PN1R0NP0L, Discrete-new:L
- added Q2, Q3: BSS138W-7-F, Discrete-new:MOSFET-N'SI1304BDL'
- added Q4: MMBT2907A, Discrete-new:TRANSISTOR-PNP
- added R101: DNP, Discrete-new:RES-0402
- added R115, R95: 22R, Discrete-new:RES-0402
- added R116, R117, R118, R23: 0R, Discrete-new:RES-0402
- added R76: 51k 1%, Discrete-new:RES-0402
- added TP10, TP34: (no value), Discrete-new:TEST-POINT-D65/35
- added U14: ESD-RCLAMP0524P, Discrete-new:ESD-RCLAMP0524P
- added U16: TLV62569DBVT, IC-new:PMIC-TLV62569'DBVT'
- added X1: ST3215SB32768H5HPWAA, Discrete-new:CRYSTAL-2P-3215
- ANT1, ANT2: value (none) -> RECE.20279.001E.01
- C1: value 10uF -> TLJB227M006R0500; device Discrete-new:CAP-0805 -> Discrete-new:CAP-POLAR-AVX-B
- C10, C9: value 0.1uF, 6.3V -> 10pF
- C11: value TLJB227M006R0500 -> 1nF 1000V; device Discrete-new:CAP-POLAR-AVX-B -> Discrete-new:CAP-1206
- C12: value 18pF, 50V -> 18pF 50V
- C13, C14: value 100nF -> 18pF 50V
- C15: value 10uF -> 18pF 50V; device Discrete-new:CAP-0805 -> Discrete-new:CAP-0402
- C16: value 100nF -> 100uF 16V; device Discrete-new:CAP-0402 -> Discrete-new:CAP-1210
- C17: value 100nF -> 100nF 50V; device Discrete-new:CAP-0402 -> Discrete-new:CAP-0805
- C18, C82, C83: value 10uF -> 10uF 25V
- C19: value 10uF -> 100nF 50V
- C2: value DNI -> 1uF 10V
- C20, C77, C78, C80: value 10uF -> 100nF 25V; device Discrete-new:CAP-0805 -> Discrete-new:CAP-0402
- C21: value 10uF, 10V -> 22uF 16V; device Discrete-new:CAP-0805 -> Discrete-new:CAP-1206
- C22: value 0.1uF, 6.3V -> 22uF 16V; device Discrete-new:CAP-0402 -> Discrete-new:CAP-1206
- C23: value 47pF -> 75pF 50V
- C24: value 47pF -> 100uF 16V; device Discrete-new:CAP-0402 -> Discrete-new:CAP-1210
- C25, C27, C28, C31, C34: value 47pF -> 100nF 25V
- C26, C38: value 47pF -> 1uF 10V
- C29, C30, C32, C33, C35, C36: value 47pF -> 10uF 25V; device Discrete-new:CAP-0402 -> Discrete-new:CAP-0805
- C3: value 0.1uF, 6.3V -> 47uF DNP; device Discrete-new:CAP-0402 -> Discrete-new:CAP-1206
- C37: value 47pF -> DNI
- C39, C41, C57: value 10uF -> 33pF 50V; device Discrete-new:CAP-0805 -> Discrete-new:CAP-0402
- C4, C5: value 18pF, 50V -> 10uF 25V; device Discrete-new:CAP-0402 -> Discrete-new:CAP-0805
- C40: value 10uF -> DNI; device Discrete-new:CAP-0805 -> Discrete-new:CAP-0402
- C42, C58: value 1uF -> 33pF 50V
- C43, C45, C46, C47, C49, C50, C60: value 100nF -> 33pF 50V
- C44, C61, C63, C65, C69, C76: value 100nF -> 100nF 25V
- C48, C51: value 100nF -> 47uF 25V; device Discrete-new:CAP-0402 -> Discrete-new:CAP-POLAR-ELECTRO-C
- C52: value 47uF DNP -> 33pF 50V; device Discrete-new:CAP-1206 -> Discrete-new:CAP-0402
- C53: value 47uF DNP -> 100nF 25V; device Discrete-new:CAP-1206 -> Discrete-new:CAP-0402
- C54: value 220uF -> 33pF 50V; device Discrete-new:CAP-POLAR-AVX-E -> Discrete-new:CAP-0402
- C55: value 10pF -> 33pF 50V
- C56: value 10pF -> 100nF 50V; device Discrete-new:CAP-0402 -> Discrete-new:CAP-0805
- C59: value DNP -> 33pF 50V
- C6: value 0.1uF, 6.3V -> 100nF 25V
- C62: value 1uF -> 100nF 25V; device Discrete-new:CAP-0603 -> Discrete-new:CAP-0402
- C64: value 1uF -> 100nF 25V
- C66: value .1uF, 6.3V -> 100nF 25V
- C67: value 22nF -> 220nF
- C68: value 100nF -> 100nF 50V; device Discrete-new:CAP-0603 -> Discrete-new:CAP-0805
- C7: value 18pF, 50V -> 47uF DNP; device Discrete-new:CAP-0402 -> Discrete-new:CAP-1206
- C70: value 47uF 25V -> 10uF 25V; device Discrete-new:CAP-POLAR-ELECTRO-C -> Discrete-new:CAP-0805
- C71: value 47uF 25V -> 100nF 25V; device Discrete-new:CAP-POLAR-ELECTRO-C -> Discrete-new:CAP-0402
- C72: value 220nF -> 100nF 25V
- C73: value 100nF -> 100nF 25V; device Discrete-new:CAP-0805 -> Discrete-new:CAP-0402
- C74: value DNI -> 10uF 25V; device Discrete-new:CAP-0402 -> Discrete-new:CAP-0805
- C75: value 1uF 10V -> 10uF 25V; device Discrete-new:CAP-0402 -> Discrete-new:CAP-0805
- C79: value 22uF -> 10uF 25V; device Discrete-new:CAP-POLAR-ELECTRO-B -> Discrete-new:CAP-0805
- C8: value 1nF -> 1uF 10V
- C81: value 22uF 16V -> 100nF 25V; device Discrete-new:CAP-1206 -> Discrete-new:CAP-0402
- C84: value 10uF -> 1uF; device Discrete-new:CAP-0805 -> Discrete-new:CAP-0402
- D1, D5, D6, D7, D8: value (none) -> Red
- D11, D9: value (none) -> DF2S6.8FS; device Discrete-new:LED'0603' -> Discrete-new:D-ESD-2P'DF2S6.8FS'
- D2, D3: value DF2S6.8FS -> Green; device Discrete-new:D-ESD-2P'DF2S6.8FS' -> Discrete-new:LED'0603'
- D4: value (none) -> Green
- F1: value 100mA MF-FSMF010X -> MF-FSMF010X
- IC1: value A4983 -> TPD4S012DRYR; device IC-new:TRANSLATOR-A4983 -> IC-new:TVS-TPD4S012DRYR
- IC2: value TPD4S012DRY -> TPD4S012DRYR
- J1: value (none) -> ST-USB-01H2; device Connector-new:HEADER-2P-65/35MIL -> Connector-new:MICRO-USB5+4P-320010050
- J2: value (none) -> DC-044; device Connector-new:HEADER-2P-65/35MIL -> Connector-new:POWER-JACK-DC'DC-044'
- J3: value 6p-2.54 -> ST-TF-003J; device OSD3358-SM-RED Platform:826646-6 -> Connector-new:MICRO-SD-CARD-HOLDER-9P'MICROSD-9P'
- J4: value ST-HD-010 -> 6p-2.54 DNP; device template:CONNECTOR-HDMI-19P -> OSD3358-SM-RED Platform:826646-6
- J5: value (none) -> WY-1223; device Connector-new:MICRO-SD-CARD-HOLDER-9P'MICROSD-9P' -> Connector-new:HEADER-4P-2.54MM
- J6: value DC Power Jack -> ST-HD-010; device For_Test_Albert:DC-044 -> template:CONNECTOR-HDMI-19P
- J7: value (none) -> 2510S-4P(T); device Connector-new:SCREW-TERMINAL-4P'3.5' -> Connector-new:HEADER-4P-65/35MIL
- J8: value (none) -> 2510S-4P(T); device Connector-new:MICRO-USB5+4P-320010050 -> Connector-new:HEADER-4P-65/35MIL
- JP2: value (none) -> ST-USB-003A; device SparkFun:M04PTH -> Connector-new:USB4+2P-320010007
- L1: value WPN201610MR47MT -> BLM15PD121SN1D; device Discrete-new:L-MPM201610SR33_T -> Discrete-new:INDUCTOR/FERRITE-BEAD'0402'
- L2: value 10uH -> BLM15PD121SN1D; device Discrete-new:INDUCTOR/FERRITE-BEAD5040S -> Discrete-new:INDUCTOR/FERRITE-BEAD'0402'
- L4: value WPN201610MR47MT -> BLM21PG331SN1D; device Discrete-new:L-MPM201610SR33_T -> Discrete-new:INDUCTOR/FERRITE-BEAD'0805'
- L5: value 150 Ohm 800mA -> BLM21PG331SN1D
- Q1: value MMBT2907 -> BSS138W-7-F; device Discrete-new:TRANSISTOR-PNP -> Discrete-new:MOSFET-N'SI1304BDL'
- R1: value 10K, 1% -> 1.5k 1%
- R10: value 0, 1% -> 10k
- R102, R103: value 10k -> 22R
- R104, R105: value 10k -> 2k
- R106, R108, R109, R112: value 33R -> 10k
- R107: value 33R -> 33k
- R11, R5: value 0, 1% -> 1k
- R110: value 33R -> 0.1R; device Discrete-new:RES-0402 -> Discrete-new:RES-1206
- R111: value DNP 10k -> 0.1R; device Discrete-new:RES-0402 -> Discrete-new:RES-1206
- R113: value 33R -> 100k 1%
- R114: value 1k -> 100k 1%
- R12: value 1.5K, 1% -> 1k
- R13, R26: value 1.5K, 1% -> 33R
- R14: value 22k 1% -> 33R
- R15: value 40.2K, 1% -> 33R
- R16, R25: value 0, 1% -> 33R
- R17: value DNP -> 499R
- R18: value 4.75K, 1% -> 1.5k 1%
- R19: value 10k -> 33R
- R2: value 1k -> 1.5k 1%
- R20: value 10K, 1% -> 40.2k 1%
- R21: value 499 -> 10k 1%
- R22: value 4.75K, 1% -> 33R
- R24: value 1M, 1%, DNI -> 0R
- R27: value 100K, 1% -> 33R
- R28, R29: value 0R -> 33R
- R3: value 1k -> 10k 1%
- R30: value 0R -> DNP 10k
- R31: value 22R -> 1k
- R32: value 1M, 1% -> 100K, 1%, DNI
- R33: value 0, 1% -> 100k 1%
- R34, R39, R80: value 10k -> 100k 1%
- R35, R36, R37, R38: value 1.5K, 1% -> 100k 1%
- R4: value 22R -> 10k
- R40: value 5.6K 1% -> 100k 1%
- R43, R44: value 22R -> 100k 1%
- R45, R46: value 2k -> 100k 1%
- R47: value 33k -> 0R
- R48, R97: value 10k -> 0R; device Discrete-new:RES-0402 -> Discrete-new:RES-1206
- R49, R50: value 10K -> 100k 1%
- R51: value 0R -> 1.5k 1%
- R52: value DNP -> 1.5k 1%
- R53: value 100K, 1% -> 1.5k 1%
- R54: value 10k, 1% -> 1.5k 1%
- R55: value 100K, 1% -> 1M 1%
- R56: value 100K, 1% -> 1M, 1%, DNI
- R57: value 100K, 1% -> 560k 1%
- R58, R60: value 100K, 1% -> 100k 1%
- R59: value 100K, 1% -> 49.9R 1%
- R6: value 100K, 1%, DNI -> 10k
- R61: value 100K, 1% -> 13.3k 1%
- R62: value 100K, 1% -> 10k 1%
- R63: value 100K, 1% -> 0R
- R64: value 100k -> 0R
- R65, R66: value 0.1R -> 0R; device Discrete-new:RES-1206 -> Discrete-new:RES-0402
- R67, R68, R71, R81, R82, R83: value 100K, 1% -> 10k
- R69: value 10R -> 10k 1%
- R7: value 0R -> 10k; device Discrete-new:RES-1206 -> Discrete-new:RES-0402
- R70: value 10K -> 10k 1%
- R77: value 10k -> 1.3k 1%
- R78: value 10k -> 240k 1%
- R79, R96: value 10k -> 1k
- R8: value 1K, 1% -> 10k
- R84: value 3.3k -> 10k
- R85: value 2.7k 1% -> 0R
- R86: value 10K, 1% -> DNP
- R87, R88, R89, R90, R91, R92: value 10K, 1% -> 10k
- R9: value 100k 1% -> 10k
- R93: value 510R 1% -> 10k
- R94: value 24k -> 10k
- R98: value 10K -> 10k
- R99: value 10K -> 5.6K 1%
- SW1, SW2: value (none) -> SKRPABE010
- TP1: value TPB0,65 -> (none); device OSD3358-SM-RED Platform:TPB0,65 -> discrete:PAD-TEST-POINT'4545'
- TP9: value (none) -> TPB0,65; device Discrete-new:TEST-POINT'4545' -> OSD3358-SM-RED Platform:TPB0,65
- U1: value (none) -> OSD3358-512M-BSM
- U10: value (none) -> SN74LVC2G241DCUR; device IC-new:LOGIC-SN74AUP1G125'DCK' -> IC-new:LOGIC-SN74LVC2G241
- U11: value ESD-RCLAMP0524P -> IT66121FN; device Discrete-new:ESD-RCLAMP0524P -> IC-new:TRANSFER_IT66121FN-9
- U12: value TL431 -> A4988SETTR-T; device IC-new:PMIC-CJ432'CJ432' -> IC-new:TRANSLATOR-A4983
- U13: value (none) -> ESD-RCLAMP0524P; device IC-new:LOGIC-SN74LVC1G07-DCK -> Discrete-new:ESD-RCLAMP0524P
- U2: value (none) -> SN74LVC1G07DCKR; device IC-new:TVS-TPD4S012DRYR -> IC-new:LOGIC-SN74LVC1G07-DCK
- U3: value MP1496DJ-LF-2 -> ATL431AIDBZR; device IC-new:CONVERTER-MP1496DJ -> IC-new:PMIC-CJ432'CJ432'
- U4: value APX811 -> WL1835MODGBMOCT; device IC-new:SUPERVISOR-APX811-31UGSOT -> moudle-new:MODULE-RF-WL1835MOD
- U5: value ETA3410 -> APX811-44UG-7; device IC-new:CONVERTER-ETA3410 -> IC-new:SUPERVISOR-APX811-31UGSOT
- U6: value SN74LVC2G241_DCU_8 -> TPS54302; device OSD3358-SM-RED Platform:SN74LVC2G241_DCU_8 -> IC-new:PMIC-TPS54302
- U7: value IT66121FN -> TPS2051BDGNR; device IC-new:TRANSFER_IT66121FN-9 -> IC-new:SWITCH-TPS2051B
- U8: value ETA3410 -> TLV62569DBVT; device IC-new:CONVERTER-ETA3410 -> IC-new:PMIC-TLV62569'DBVT'
- U9: value ESD-RCLAMP0524P -> SN74LVC1G125DCKR; device Discrete-new:ESD-RCLAMP0524P -> IC-new:LOGIC-SN74AUP1G125'DCK'
- Y1: value ABS07-32.768KHZ-T -> CX3225GB24000P0HPQCC; device OSD3358-SM-RED Platform:ABS07-32.768KHZ-T -> OSD3358-SM-RED Platform:7A-24.000MAAJ-T
- renumbered ANT3 to ANT2, ANT4 to ANT1, FB2 to L9, FB3 to L5, FB7 to L7, FB8 to L8, IC15 to IC2
Connections:
- removed net N$14: C67.2, U3.SS
- removed net N$26: L1.1, U5.SW
- removed net N$3: C65.2, U3.VCC
- removed net N$53: R14.2, R9.1, U5.FB
- removed net N$66: R69.1, U3.BS
- removed net N$68: C76.1, L2.1, U3.SW
- removed net N$71: C76.2, R69.2
- removed net N$73: R84.1, U3.FB
- removed net N$74: C59.2, R84.2, R85.2, R93.2
- removed net N$78: R64.1, R94.1, U3.EN/SYNC
- new net N$77: R76.2, R78.2, U8.FB
- new net N$79: L6.1, U8.SW
- new net N$80: R76.1, R77.2
- new net N$84: R57.1, R58.2, U6.EN
- new net N$86: C19.2, U6.BOOT
- new net N$87: C19.1, L3.1, U6.SW
- new net N$88: C23.1, R59.1, R60.2
- new net N$89: C23.2, R60.1, R61.2, U6.FB
- net 1.8V-WIFI: now also C2.1, C7.2, C8.1, L1.2, R10.1, R30.1, R4.1, R6.1, R7.1, R8.1, R9.1, U4.VIO; no longer C52.2, C58.1, C64.1, FB6.2, MOD1.VIO, R100.1, R102.1, R103.1, R104.1, R111.1, R96.1, R97.1
- net 12VDC: now also C48.+, C51.+, C68.2, R97.2, U12.VBB1, U12.VBB2; no longer C70.+, C71.+, C73.2, IC1.VBB1, IC1.VBB2, R7.2
- net 3.3V-WIFI: now also C3.2, C4.1, C5.1, C6.1, L2.2, R11.2, R12.2, R5.2, U4.VBAT_IN1, U4.VBAT_IN2; no longer C39.1, C53.2, C57.1, C63.1, FB1.2, MOD1.VBAT_IN1, MOD1.VBAT_IN2, R114.2, R124.2, R125.2
- net AGND: now also C25.2, C27.2, C28.2, R66.2; no longer C10.2, C8.2, C9.2, R25.2
- net BT_EN: now also Q3.G, U4.BT_EN; no longer MOD1.BT_EN, T4.G
- net BT_HCI_CTS: now also R14.2; no longer R141.2
- net BT_HCI_RTS: now also R13.2; no longer R140.2
- net BT_HCI_RX: now also R16.2; no longer R143.2
- net BT_HCI_TX: now also R15.2; no longer R142.2
- net B_UART0_RX: now also J4.4, R80.2, U10.1A; no longer J3.4, R27.2, U6.1A
- net B_UART0_TX: now also J4.5, U10.2Y; no longer J3.5, U6.2Y
- net CEC: now also D12.2, J6.CE_REMOTE, R106.2, U11.CEC; no longer D10.2, J4.CE_REMOTE, R48.2, U7.CEC
- net CGND: now also C11.2, J1.GND@1, J1.GND@2, J1.GND@3, J1.GND@4, J3.G2, J6.SHELL3, J6.SHELL4, JP2.GND@1, JP2.GND@2, R48.2; no longer J5.G2, J5.G3, J8.GND@1, J8.GND@2, J8.GND@3, J8.GND@4, X2.CG1, X2.CG2
- net CK_N: now also J6.CK-, U11.TXCM, U14.5, U14.6; no longer J4.CK-, U7.TXCM, U9.5, U9.6
- net CK_P: now also J6.CK+, U11.TXCP, U14.4, U14.7; no longer J4.CK+, U7.TXCP, U9.4, U9.7
- net CLKOUT2: now also C37.2, R79.2, R96.2, U4.EXT_32K; no longer C2.2, MOD1.EXT_32K, R2.2, R3.2
- net COILA+: now also J5.P$1, U12.OUT1B; no longer IC1.OUT1B, J7.4, JP3.4, JP5.4
- net COILA-: now also J5.P$2, U12.OUT1A; no longer IC1.OUT1A, J7.3, JP3.3, JP5.3
- net COILB+: now also J5.P$4, U12.OUT2B; no longer IC1.OUT2B, J7.1, JP3.1, JP5.1
- net COILB-: now also J5.P$3, U12.OUT2A; no longer IC1.OUT2A, J7.2, JP3.2, JP5.2
- net CUR_REF: now also U12.REF; no longer IC1.REF, TP33.TP
- net D0_N: now also J6.D0-, U11.TX0M, U14.2, U14.9; no longer J4.D0-, U7.TX0M, U9.2, U9.9
- net D0_P: now also J6.D0+, U11.TX0P, U14.1, U14.10; no longer J4.D0+, U7.TX0P, U9.1, U9.10
- net D1_N: now also J6.D1-, U11.TX1M, U13.5, U13.6; no longer J4.D1-, U11.5, U11.6, U7.TX1M
- net D1_P: now also J6.D1+, U11.TX1P, U13.4, U13.7; no longer J4.D1+, U11.4, U11.7, U7.TX1P
- net D2_N: now also J6.D2-, U11.TX2M, U13.2, U13.9; no longer J4.D2-, U11.2, U11.9, U7.TX2M
- net D2_P: now also J6.D2+, U11.TX2P, U13.1, U13.10; no longer J4.D2+, U11.1, U11.10, U7.TX2P
- net DDC_SCL: now also D9.2, J6.DDC_CLK, R102.2, R104.2; no longer D12.2, J4.DDC_CLK, R43.2, R45.2
- net DDC_SDA: now also D10.2, J6.DDC_DATA, R103.2, R105.2; no longer D2.2, J4.DDC_DATA, R44.2, R46.2
- net DIR(GPIO23): now also R88.1, U12.DIR; no longer IC1.DIR, R78.1
- net EEPROM_WP: now also TP10.T; no longer J1.1
- net ENABLE(GPIO46): now also R94.1, U12.ENABLE; no longer IC1.ENABLE, R77.1
- net GND: now also C1.-, C11.1, C2.2, C20.2, C21.1, C22.1, C26.1, C29.1, C3.1, C30.1, C33.1, C35.1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; no longer C1.1, C11.-, C13.1, C14.1, C15.1, C19.1, C2.1, C20.1, C21.2, C22.2, C23.2, C25.2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
- net HDMI_1V2: now also C61.2, C62.2, C63.2, C64.2, C65.2, C66.2, C82.2, C83.2, L10.2, R113.2, U11.AVCC12, U11.DVDD12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; no longer C19.2, C40.2, C43.2, C44.2, C45.2, C46.2, C47.2, C48.2, L4.2, R41.2, U7.AVCC12, U7.DVDD12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
- net HDMI_3V3: now also C69.2, C71.2, C73.2, C76.2, C77.2, C78.2, R100.1, R106.1, R109.2, R81.1, R82.1, R83.1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; no longer C17.2, C49.2, C50.2, C51.2, C60.2, C61.2, R105.2, R34.1, R48.1, R49.1, R50.1, R98.1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
- net HDMI_5V: now also C84.2, D11.2, J6.+5V, R104.1, R105.1; no longer C42.2, D3.2, J4.+5V, R45.1, R46.1
- net HDMI_AUDBCLK: now also U11.SCK/MCLK; no longer U7.SCK/MCLK
- net HDMI_AUDDOUT: now also R85.1, R86.1; no longer R51.1, R52.1
- net HDMI_AUDWCLK: now also U11.WS; no longer U7.WS
- net HDMI_INT: now also R83.2, U11.INT; no longer R50.2, U7.INT
- net HDMI_NRST: now also C38.2, R84.2, U11.SYSRSTN; no longer C62.2, R49.2, U7.SYSRSTN
- net HPD: now also J6.HPD, R107.2, U11.HPD; no longer J4.HPD, R47.2, U7.HPD
- net I2C0_SCL: now also R1.1; no longer R12.1
- net I2C0_SDA: now also R2.1; no longer R13.1
- net I2C2_SCL: now also R82.2, U11.PCSCL; no longer R98.2, U7.PCSCL
- net I2C2_SDA: now also R81.2, U11.PCSDA; no longer R99.2, U7.PCSDA
- net LCD_DATA0: now also C60.1, R50.2, U11.D3; no longer C38.1, R68.2, U7.D3
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Other:
- note added: "I = 100mA"
- note added: "I = 1A"
- note added: "I = 200mA"
- note added: "I = 2A"
- note added: "I = 3A"
- note added: "I = 500mA"
- note added: "Vout=0.6Vx(1+R1/R2)"
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
Commit message: Latest from Seeed
Parts:
- added R119: 10k, Discrete-new:RES-0402
- C84: value 1uF -> 1uF 10V
- R63: value 0R -> 10k
Connections:
- removed net AIN0: U1B.AIN0
- removed net AIN1: U1B.AIN1
- removed net AIN2: U1B.AIN2
- removed net AIN3: U1B.AIN3
- removed net AIN4: U1B.AIN4
- removed net AIN5: U1B.AIN5
- removed net AIN6: U1B.AIN6
- removed net JTAG_EMU0: U1B.EMU0
- removed net JTAG_EMU1: U1B.EMU1
- removed net JTAG_TCK: U1B.TCK
- removed net JTAG_TDI: U1B.TDI
- removed net JTAG_TDO: U1B.TDO
- removed net JTAG_TMS: U1B.TMS
- removed net JTAG_TRSTN: U1B.TRSTN
- net BT_HCI_CTS: now also U1D.MDC; no longer U1D.MDIO
- net BT_HCI_RTS: now also U1D.MDIO; no longer U1D.MDC
- net BT_HCI_RX: now also U1D.MII1_RXD2; no longer U1D.MII1_RXD3
- net BT_HCI_TX: now also U1D.MII1_RXD3; no longer U1D.MII1_RXD2
- net CGND: now also J3.G3, J6.SHELL1, J6.SHELL2
- net GND: now also R119.2
- net N$32: now also R119.1
Other:
- moved on the sheet: TP25
